File: Flight-Controller-PCB1/flight-controller.sch (EAGLE design)
At the start: 2 parts

Commit message: added board libraries and board file
Parts:
- added 3X3MM1: CURRENT_BOOTLOADERLQFP-32, Teensy_DIY_v1.0:CURRENT_BOOTLOADERLQFP-32
- added U$3: LP38691DT, national_lp38691:LP38691DT
- U$1: value TEENSY_3.1_ALL_PINS_AND_PADS -> MK20DX256VLH7; device Teensy_3_and_LC_Series_Boards_v1.0:TEENSY_3.1_ALL_PINS_AND_PADS -> Teensy_DIY_v1.0:MK20DX256VLH7
Connections:
- new net N$1: 3X3MM1.PTA7, U$1.D0/RX1/TOUCH
Changed lines of the file:
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@@
 <layer number="54" name="bGND_GNDA" color="1" fill="9" visible="no" active="no"/>
 <layer number="56" name="wert" color="7" fill="1" visible="no" active="no"/>
+<layer number="57" name="tCAD" color="7" fill="1" visible="no" active="no"/>
 <layer number="90" name="Modules" color="5" fill="1" visible="yes" active="yes"/>
 <layer number="91" name="Nets" color="2" fill="1" visible="yes" active="yes"/>
@@
 <layer number="97" name="Info" color="7" fill="1" visible="yes" active="yes"/>
 <layer number="98" name="Guide" color="6" fill="1" visible="yes" active="yes"/>
+<layer number="99" name="SpiceOrder" color="7" fill="1" visible="yes" active="yes"/>
 <layer number="100" name="Muster" color="7" fill="1" visible="no" active="no"/>
 <layer number="101" name="Patch_Top" color="12" fill="4" visible="yes" active="yes"/>
 <layer number="102" name="Vscore" color="7" fill="1" visible="yes" active="yes"/>
+<layer number="103" name="fp3" color="7" fill="1" visible="no" active="yes"/>
 <layer number="104" name="Name" color="7" fill="1" visible="yes" active="yes"/>
+<layer number="105" name="Beschreib" color="9" fill="1" visible="yes" active="yes"/>
+<layer number="106" name="BGA-Top" color="4" fill="1" visible="yes" active="yes"/>
+<layer number="107" name="BD-Top" color="5" fill="1" visible="yes" active="yes"/>
+<layer number="108" name="fp8" color="7" fill="1" visible="no" active="yes"/>
+<layer number="109" name="fp9" color="7" fill="1" visible="no" active="yes"/>
+<layer number="110" name="fp0" color="7" fill="1" visible="no" active="yes"/>
+<layer number="111" name="LPC17xx" color="7" fill="1" visible="yes" active="yes"/>
+<layer number="112" name="tSilk" color="7" fill="1" visible="yes" active="yes"/>
+<layer number="113" name="IDFDebug" color="7" fill="1" visible="yes" active="yes"/>
 <layer number="116" name="Patch_BOT" color="9" fill="4" visible="yes" active="yes"/>
+<layer number="117" name="mPads" color="7" fill="1" visible="no" active="no"/>
+<layer number="118" name="mVias" color="7" fill="1" visible="no" active="no"/>
+<layer number="119" name="mUnrouted" color="7" fill="1" visible="no" active="no"/>
+<layer number="120" name="mDimension" color="7" fill="1" visible="no" active="no"/>
 <layer number="121" name="_tsilk" color="7" fill="1" visible="yes" active="yes"/>
 <layer number="122" name="_bsilk" color="7" fill="1" visible="yes" active="yes"/>
+<layer number="123" name="tTestmark" color="7" fill="1" visible="no" active="yes"/>
+<layer number="124" name="bTestmark" color="7" fill="1" visible="no" active="yes"/>
+<layer number="125" name="_tNames" color="7" fill="1" visible="yes" active="yes"/>
+<layer number="126" name="_bNames" color="7" fill="1" visible="yes" active="yes"/>
+<layer number="127" name="_tValues" color="7" fill="1" visible="yes" active="yes"/>
+<layer number="128" name="_bValues" color="7" fill="1" visible="yes" active="yes"/>
+<layer number="129" name="mtStop" color="7" fill="1" visible="no" active="no"/>
+<layer number="130" name="mbStop" color="7" fill="1" visible="no" active="no"/>
+<layer number="131" name="tAdjust" color="7" fill="1" visible="no" active="yes"/>
+<layer number="132" name="bAdjust" color="7" fill="1" visible="no" active="yes"/>
+<layer number="133" name="mtFinish" color="7" fill="1" visible="no" active="no"/>
+<layer number="134" name="mbFinish" color="7" fill="1" visible="no" active="no"/>
+<layer number="135" name="mtGlue" color="7" fill="1" visible="no" active="no"/>
+<layer number="136" name="mbGlue" color="7" fill="1" visible="no" active="no"/>
+<layer number="137" name="mtTest" color="7" fill="1" visible="no" active="no"/>
+<layer number="138" name="mbTest" color="7" fill="1" visible="no" active="no"/>
+<layer number="139" name="mtKeepout" color="7" fill="1" visible="no" active="no"/>
+<layer number="140" name="mbKeepout" color="7" fill="1" visible="no" active="no"/>
+<layer number="141" name="mtRestrict" color="7" fill="1" visible="no" active="no"/>
+<layer number="142" name="mbRestrict" color="7" fill="1" visible="no" active="no"/>
+<layer number="143" name="mvRestrict" color="7" fill="1" visible="no" active="no"/>
+<layer number="144" name="Drill_legend" color="7" fill="1" visible="yes" active="yes"/>
+<layer number="145" name="mHoles" color="7" fill="1" visible="no" active="no"/>
+<layer number="146" name="mMilling" color="7" fill="1" visible="no" active="no"/>
+<layer number="147" name="mMeasures" color="7" fill="1" visible="no" active="no"/>
+<layer number="148" name="mDocument" color="7" fill="1" visible="no" active="no"/>
+<layer number="149" name="mReference" color="7" fill="1" visible="no" active="no"/>
+<layer number="150" name="Notes" color="7" fill="1" visible="no" active="yes"/>
 <layer number="151" name="HeatSink" color="7" fill="1" visible="yes" active="yes"/>
+<layer number="152" name="_bDocu" color="7" fill="1" visible="yes" active="yes"/>
+<layer number="153" name="FabDoc1" color="6" fill="1" visible="no" active="no"/>
+<layer number="154" name="FabDoc2" color="2" fill="1" visible="no" active="no"/>
+<layer number="155" name="FabDoc3" color="7" fill="15" visible="no" active="no"/>
+<layer number="191" name="mNets" color="7" fill="1" visible="no" active="no"/>
+<layer number="192" name="mBusses" color="7" fill="1" visible="no" active="no"/>
+<layer number="193" name="mPins" color="7" fill="1" visible="no" active="no"/>
+<layer number="194" name="mSymbols" color="7" fill="1" visible="no" active="no"/>
+<layer number="195" name="mNames" color="7" fill="1" visible="no" active="no"/>
+<layer number="196" name="mValues" color="7" fill="1" visible="no" active="no"/>
+<layer number="199" name="Contour" color="7" fill="1" visible="yes" active="yes"/>
 <layer number="200" name="200bmp" color="1" fill="10" visible="yes" active="yes"/>
 <layer number="201" name="201bmp" color="2" fill="10" visible="yes" active="yes"/>
@@
 <layer number="207" name="207bmp" color="8" fill="10" visible="yes" active="yes"/>
 <layer number="208" name="208bmp" color="9" fill="10" visible="yes" active="yes"/>
+<layer number="209" name="209bmp" color="7" fill="1" visible="no" active="yes"/>
+<layer number="210" name="210bmp" color="7" fill="1" visible="no" active="yes"/>
+<layer number="211" name="211bmp" color="7" fill="1" visible="yes" active="yes"/>
+<layer number="212" name="212bmp" color="7" fill="1" visible="yes" active="yes"/>
+<layer number="213" name="213bmp" color="7" fill="1" visible="yes" active="yes"/>
+<layer number="214" name="214bmp" color="7" fill="1" visible="yes" active="yes"/>
+<layer number="215" name="215bmp" color="7" fill="1" visible="yes" active="yes"/>
+<layer number="216" name="216bmp" color="7" fill="1" visible="yes" active="yes"/>
+<layer number="217" name="217bmp" color="18" fill="1" visible="no" active="no"/>
+<layer number="218" name="218bmp" color="19" fill="1" visible="no" active="no"/>
+<layer number="219" name="219bmp" color="20" fill="1" visible="no" active="no"/>
+<layer number="220" name="220bmp" color="21" fill="1" visible="no" active="no"/>
+<layer number="221" name="221bmp" color="22" fill="1" visible="no" active="no"/>
+<layer number="222" name="222bmp" color="23" fill="1" visible="no" active="no"/>
+<layer number="223" name="223bmp" color="24" fill="1" visible="no" active="no"/>
+<layer number="224" name="224bmp" color="25" fill="1" visible="no" active="no"/>
+<layer number="248" name="Housing" color="7" fill="1" visible="yes" active="yes"/>
+<layer number="249" name="Edge" color="7" fill="1" visible="yes" active="yes"/>
 <layer number="250" name="Descript" color="3" fill="1" visible="no" active="no"/>
 <layer number="251" name="SMDround" color="12" fill="11" visible="no" active="no"/>
@@
 </classes>
 <parts>
-<part name="U$1" library="Teensy_3_and_LC_Series_Boards_v1.0" deviceset="TEENSY_3.1_ALL_PINS_AND_PADS" device=""/>
 <part name="U$2" library="con-hirose" deviceset="MICRO-USB-" device="ZX62R-B-5P"/>
+<part name="3X3MM1" library="Teensy_DIY_v1.0" deviceset="CURRENT_BOOTLOADER" device="LQFP-32"/>
+<part name="U$3" library="national_lp38691" deviceset="LP38691DT" device=""/>
+<part name="U$1" library="Teensy_DIY_v1.0" deviceset="MK20DX256VLH7" device=""/>
 </parts>
 <sheets>
@@
 </plain>
 <instances>
-<instance part="U$1" gate="G$1" x="129.54" y="50.8"/>
 <instance part="U$2" gate="G$1" x="-12.7" y="50.8"/>
+<instance part="3X3MM1" gate="G$1" x="40.64" y="15.24"/>
+<instance part="U$3" gate="G$1" x="40.64" y="91.44"/>
+<instance part="U$1" gate="G$1" x="116.84" y="58.42" rot="R180"/>
 </instances>
 <busses>
 </busses>
 <nets>
+<net name="N$1" class="0">
+<segment>
+<pinref part="3X3MM1" gate="G$1" pin="PTA7"/>
+<pinref part="U$1" gate="G$1" pin="D0/RX1/TOUCH"/>
+<wire x1="144.78" y1="7.62" x2="55.88" y2="20.32" width="0.1524" layer="91"/>
+</segment>
+</net>
 </nets>
 </sheet>

Commit message: updated project file
Parts:
- removed 3X3MM1: CURRENT_BOOTLOADERLQFP-32, Teensy_DIY_v1.0:CURRENT_BOOTLOADERLQFP-32
- removed U$1: MK20DX256VLH7, Teensy_DIY_v1.0:MK20DX256VLH7
- removed U$2: MICRO-USB-ZX62R-B-5P, con-hirose:MICRO-USB-ZX62R-B-5P
- removed U$3: LP38691DT, national_lp38691:LP38691DT
- added C1: 10uF, appfruits:CAPACITOR-10UF
- added C11, C14, C16, C18, C19, C2, C21, C22, C4, C5: 0.1uF, appfruits:CAPACITOR-0.1UF
- added C17, C20: 2.2uF, appfruits:CAPACITOR-2.2UF
- added C3: 22uF, appfruits:CAPACITOR-22UF
- added J1: 1981584-1, con-usb:1981584-1
- added L1: 2.2uH, 2.1A, appfruits:LPS30152.2UH
- added L2, L3, L4: 600 Ohm/100 Mhz, appfruits:INDUCTOR-BK2125HM601-T
- added LED: AMBER/ 592 nm, appfruits:LED-AMBER
- added LED1: (no value), appfruits:LED-GREEN
- added PROGRAM: Program, SparkFun-Electromechanical:SWITCH-MOMENTARY-2-SMD-1101NE
- added R10: 1K, appfruits:RESISTOR-1K
- added R16, R30, R9: 470, appfruits:RESISTOR-470
- added R2: 10K, appfruits:RESISTOR-10K
- added R3: 2M, appfruits:RESISTOR-2M
- added R4, R6: 220K, appfruits:RESISTOR-220K
- added R7: 1.2M, appfruits:RESISTOR-1.2M
- added RN1: 33, resistor-dil:2R-NEXB34V
- added U1: MK20DX256VLH7, appfruits:MK20DX256VLH7
- added U2: TPS61200, appfruits:TPS61200
- added U3: MINI54TAN, TeensyCustom:MINI54TAN
- added Y1: 32.768KHz, appfruits:CRYSTAL/32.768KHZ/SMD-TXC_7A
- added Y2: 16Mhz/8pF, appfruits:CRYSTAL/SMD-5X3-GND16MHZ/8PF
Connections:
- new net 3.3V: C18.1, C19.1, C20.1, C21.1, C22.1, C3.1, C5.1, L3.2, LED1.C, R7.2, U1.VBAT, U1.VDD, U1.VOUT33, U1.VREGIN, U2.VOUT, U3.AVDD, U3.VDD
- new net FB: R6.2, R7.1, U2.FB
- new net GND: C14.2, C18.2, C19.2, C20.2, C21.2, C22.2, C5.2, J1.GND, L2.1, L4.1, PROGRAM.1, R30.1, R4.1, R6.1, R9.2, U1.VSS, U3.AVSS, U3.P1.4, U3.P2.5, U3.VSS
- new net ID: J1.ID, U1.PTA1, U3.P0.0
- new net MISO: U1.PTC7
- new net MOSI: U1.PTC6
- new net N$12: LED.A, U1.PTC8
- new net N$15: U1.PTA2, U3.P0.1
- new net N$18: LED.C, R30.2
- new net N$19: PROGRAM.2, U3.P5.2
- new net N$2: L1.1, U2.L
- new net N$22: C14.1, U3.LDOCAP
- new net N$27: U1.PTA18, Y2G$1.2
- new net N$28: U1.PTA19, Y2G$1.1
- new net N$29: U1.XTAL32, Y1.2
- new net N$30: U1.EXTAL32, Y1.1
- new net PGND: C1.2, C3.2, C4.2, U2.GND, U2.PAD@1, U2.PAD@2, U2.PAD@3, U2.PAD@4, U2.PAD@5, U2.PGND
- new net PS: R2.2, U2.PS
- new net RESET_B: U1.RESET_B, U3.P3.2
- new net SCK: U1.PTC5
- new net SCL: U1.PTB2
- new net SDA: U1.PTB3
- new net SOFTPOWER: R10.1, U2.EN
- new net SWD_CLK: U1.PTA0, U3.P0.7
- new net SWD_DIO: U1.PTA3, U3.P0.5, U3.P0.6
- new net USB_CON_N: J1.D-, RN1A.1
- new net USB_CON_P: J1.D+, RN1B.1
- new net USB_D_N: RN1A.2, U1.USB0_DM
- new net USB_D_P: RN1B.2, U1.USB0_DP
- new net USB_SHIELD: J1.S1, J1.S2, J1.S3, J1.S4, L2.2
- new net UVLO: C2.2, R3.1, R4.2, U2.UVLO
- new net VAUX: C4.1, U2.VAUX
- new net VCC: C1.1, C2.1, J1.VBUS, L1.2, R10.2, R2.1, R3.2, U2.VIN
- new net VDDA: C17.1, L3.1, R16.1, U1.VDDA
- new net VREFH: C11.1, R16.2, U1.VREFH
- new net VREFL: C11.2, C16.2, C17.2, L4.2, U1.VREFL, U1.VSSA
- new net VREF_OUT: C16.1, U1.VREF_OUT
- net N$1: now also LED1.A, R9.1; no longer 3X3MM1.PTA7, U$1.D0/RX1/TOUCH
Other:
- note added: "If you don't want to waste energy remove this power led as all it does is indicating applied power."
- note added: "MCU"
- note added: "MCU based on the amazing Teensy 3.1, developed by Paul J Stoffregen and pjrc.com."
- note added: "Parts of this these schematics were inspired/taken from Teensy 3.1 schematics published by Paul J. Stoffregen at www.pjrc.com and Sparkfuns Power Cell schematics (https://www.sparkfun.com/products/11231) These schematics have been successfully working in a real world project and are provided as a reference for your own custom board."
- note added: "Place RN1 as close as possible to USB-Connector!"
- note added: "Published June 2015 by Phillip Schuster (www.appfruits.com)"
- note added: "Released under the Creative Commons Attribution Share-Alike 4.0 License https://creativecommons.org/licenses/by-sa/4.0/"
- note added: "Switching Regulator"
- note added: "Switchting regulator 3.3V based on Sparkfuns Power Cell Schematics: https://www.sparkfun.com/products/11231"
- note added: "This switching regulator has been used in a LIPO based project. If you are running your board only USB-connected this circuit is overkill, use a simple 3.3V Low dropout regulator in a SOC 223 package for easier soldering and board layout. But it's important to get a clean, noise free 3.3V power supply and it should be able to provide a minimum of 150mA (this circuit is able to provide 300 mA)"
- note added: "USB-Connector"
- note added: "USB_D+ and USB_D- must be routed as a differential pair. By naming them with _N and _P Eagle automatically routes both traces when placing traces in board layout. It uses the DRU and/or net class values. See EAGLE-Menu Edit->Net classes for the values in this example board"
- note added: "UVLO 2.6V"
