File: Flight-Controller-PCB1/flight-controller.sch (EAGLE design)
At the start: 45 parts, among them J1 1981584-1, U1 MK20DX256VLH7, U2 TPS61200, U3 MINI54TAN, Y1 32.768KHz, Y2 16Mhz/8pF

Commit message: working on arduino pro mini
Parts:
- added C12, C13: 0.1uF, SparkFun:CAP0603-CAP
- added D3: Green, Testing:LED
- added JP1: FTDI Basic, SparkFun:ARDUINO_SERIAL_PROGRAMPTH
- added Q1: 8/16/20MHz, Testing:RESONATOR1:1
- added R11: 330, SparkFun:RESISTOR0603-RES
- added R12, R13: (no value), SparkFun:RESISTOR0603-RES
- added R8: 10K, SparkFun:RESISTOR0603-RES
- added S1: Reset, Testing:SWITCH-MOMENTARY-2SMD-ALT01
- added U4: ATMEGA328, SparkFun:ATMEGA168
Connections:
- new net A4: R12.1, U4.PC4(ADC4/SDA)
- new net A5: R13.1, U4.PC5(ADC5/SCL)
- new net AREF: C12.2, U4.AREF
- new net DTR: C13.2, JP1.DTR
- new net N$6: Q1.3, U4.PB7(XTAL2/TOSC2)
- new net N$7: D3.A, R11.2
- new net N$8: Q1.1, U4.PB6(XTAL1/TOSC1)
- new net RESET: C13.1, R8.1, S1.2, U4.PC6(/RESET)
- new net RXI: JP1.TXO
- new net TXO: JP1.RXI
- net 3.3V: now also R12.2, R13.2, R8.2, U4.AVCC, U4.VCC@1, U4.VCC@2
- net GND: now also C12.1, D3.C, JP1.CTS, JP1.GND, Q1.2, S1.1, U4.AGND, U4.GND@1, U4.GND@2
- net SCK: now also R11.1, U4.PB5(SCK)
- net VCC: now also JP1.VCC
Other:
- note removed: "MCU"
- note removed: "MCU based on the amazing Teensy 3.1, developed by Paul J Stoffregen and pjrc.com."

Commit message: still working on microcontroller
Connections:
- removed net RXI: JP1.TXO
- removed net TXO: JP1.RXI
- new net N$10: JP1.RXI, U4.PD1(TXD)
- new net N$9: JP1.TXO, U4.PD0(RXD)
- net 3.3V: now also JP1.VCC
- net VCC: no longer JP1.VCC
Changed lines of the file:
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@@
 <wire x1="0" y1="124.46" x2="246.38" y2="124.46" width="0.4064" layer="97" style="shortdash"/>
 <wire x1="246.38" y1="124.46" x2="246.38" y2="68.58" width="0.4064" layer="97" style="shortdash"/>
-<wire x1="246.38" y1="68.58" x2="246.38" y2="-15.24" width="0.4064" layer="97" style="shortdash"/>
 <wire x1="0" y1="68.58" x2="246.38" y2="68.58" width="0.4064" layer="97" style="shortdash"/>
-<wire x1="246.38" y1="-15.24" x2="246.38" y2="-220.98" width="0.4064" layer="97" style="shortdash"/>
+<wire x1="246.38" y1="68.58" x2="246.38" y2="-220.98" width="0.4064" layer="97" style="shortdash"/>
 <wire x1="0" y1="-220.98" x2="246.38" y2="-220.98" width="0.4064" layer="97" style="shortdash"/>
 <wire x1="0" y1="124.46" x2="0" y2="68.58" width="0.4064" layer="97" style="shortdash"/>
@@
 </instance>
 <instance part="JP1" gate="G$1" x="-20.32" y="-165.1"/>
-<instance part="U$11" gate="G$1" x="-40.64" y="-48.26"/>
-<instance part="U$13" gate="G$1" x="15.24" y="-48.26"/>
-<instance part="U$15" gate="G$1" x="22.86" y="-48.26"/>
-<instance part="U$16" gate="G$1" x="-63.5" y="-35.56"/>
+<instance part="U$11" gate="G$1" x="-40.64" y="-45.72"/>
+<instance part="U$13" gate="G$1" x="15.24" y="-45.72"/>
+<instance part="U$15" gate="G$1" x="22.86" y="-45.72"/>
+<instance part="U$16" gate="G$1" x="-63.5" y="-25.4"/>
 </instances>
 <busses>
@@
 </segment>
 <segment>
-<wire x1="-40.64" y1="-58.42" x2="-40.64" y2="-50.8" width="0.1524" layer="91"/>
+<wire x1="-40.64" y1="-58.42" x2="-40.64" y2="-48.26" width="0.1524" layer="91"/>
 <wire x1="-40.64" y1="-63.5" x2="-40.64" y2="-60.96" width="0.1524" layer="91"/>
 <wire x1="-40.64" y1="-60.96" x2="-40.64" y2="-58.42" width="0.1524" layer="91"/>
@@
 </segment>
 <segment>
-<wire x1="15.24" y1="-53.34" x2="15.24" y2="-50.8" width="0.1524" layer="91"/>
+<wire x1="15.24" y1="-53.34" x2="15.24" y2="-48.26" width="0.1524" layer="91"/>
 <pinref part="R12" gate="G$1" pin="2"/>
 <pinref part="U$13" gate="G$1" pin="3.3V"/>
 </segment>
 <segment>
-<wire x1="22.86" y1="-55.88" x2="22.86" y2="-50.8" width="0.1524" layer="91"/>
+<wire x1="22.86" y1="-55.88" x2="22.86" y2="-48.26" width="0.1524" layer="91"/>
 <pinref part="R13" gate="G$1" pin="2"/>
 <pinref part="U$15" gate="G$1" pin="3.3V"/>
 </segment>
 <segment>
-<wire x1="-63.5" y1="-38.1" x2="-63.5" y2="-40.64" width="0.1524" layer="91"/>
+<wire x1="-63.5" y1="-27.94" x2="-63.5" y2="-40.64" width="0.1524" layer="91"/>
 <pinref part="R8" gate="G$1" pin="2"/>
 <pinref part="U$16" gate="G$1" pin="3.3V"/>
+<pinref part="JP1" gate="G$1" pin="VCC"/>
+<wire x1="-15.24" y1="-162.56" x2="-2.54" y2="-162.56" width="0.1524" layer="91"/>
+<wire x1="-2.54" y1="-162.56" x2="-2.54" y2="-147.32" width="0.1524" layer="91"/>
+<wire x1="-2.54" y1="-147.32" x2="-101.6" y2="-147.32" width="0.1524" layer="91"/>
+<wire x1="-101.6" y1="-147.32" x2="-101.6" y2="-40.64" width="0.1524" layer="91"/>
+<wire x1="-101.6" y1="-40.64" x2="-63.5" y2="-40.64" width="0.1524" layer="91"/>
 </segment>
 </net>
@@
 <pinref part="SUPPLY1" gate="G$1" pin="VCC"/>
 </segment>
-<segment>
-<wire x1="-15.24" y1="-162.56" x2="-12.7" y2="-162.56" width="0.1524" layer="91"/>
-<pinref part="JP1" gate="G$1" pin="VCC"/>
-<label x="-12.7" y="-162.56" size="1.27" layer="95" xref="yes"/>
-</segment>
 </net>
 <net name="N$12" class="0">
@@
 </segment>
 </net>
-<net name="TXO" class="0">
-<segment>
-<wire x1="-15.24" y1="-167.64" x2="-12.7" y2="-167.64" width="0.1524" layer="91"/>
+<net name="N$9" class="0">
+<segment>
+<pinref part="JP1" gate="G$1" pin="TXO"/>
+<wire x1="-15.24" y1="-165.1" x2="20.32" y2="-165.1" width="0.1524" layer="91"/>
+<wire x1="20.32" y1="-165.1" x2="20.32" y2="-76.2" width="0.1524" layer="91"/>
+<pinref part="U4" gate="G$1" pin="PD0(RXD)"/>
+<wire x1="20.32" y1="-76.2" x2="7.62" y2="-76.2" width="0.1524" layer="91"/>
+</segment>
+</net>
+<net name="N$10" class="0">
+<segment>
 <pinref part="JP1" gate="G$1" pin="RXI"/>
-<label x="-12.7" y="-167.64" size="1.27" layer="95" xref="yes"/>
-</segment>
-</net>
-<net name="RXI" class="0">
-<segment>
-<wire x1="-15.24" y1="-165.1" x2="-12.7" y2="-165.1" width="0.1524" layer="91"/>
-<pinref part="JP1" gate="G$1" pin="TXO"/>
-<label x="-12.7" y="-165.1" size="1.27" layer="95" xref="yes"/>
-</segment>
-</net>
+<wire x1="-15.24" y1="-167.64" x2="22.86" y2="-167.64" width="0.1524" layer="91"/>
+<wire x1="22.86" y1="-167.64" x2="22.86" y2="-78.74" width="0.1524" layer="91"/>
+<pinref part="U4" gate="G$1" pin="PD1(TXD)"/>
+<wire x1="22.86" y1="-78.74" x2="7.62" y2="-78.74" width="0.1524" layer="91"/>
+</segment>
+</net>

Commit message: laying out board for final time
Parts:
- removed R12, R13: (no value), SparkFun:RESISTOR0603-RES
Connections:
- removed net A4: R12.1, U4.PC4(ADC4/SDA)
- removed net A5: R13.1, U4.PC5(ADC5/SCL)
- new net NONE: R11.1, U4.PB5(SCK)
- net 3.3V: no longer R12.2, R13.2
- net SCK: no longer R11.1, U4.PB5(SCK)
- net SCL: now also U4.PC5(ADC5/SCL)
- net SDA: now also U4.PC4(ADC4/SDA)
Changed lines of the file:
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@@
 <?xml version="1.0" encoding="utf-8"?>
 <!DOCTYPE eagle SYSTEM "eagle.dtd">
-<eagle version="7.5.0">
+<eagle version="7.4.0">
 <drawing>
 <settings>
@@
 <part name="GND19" library="SparkFun" deviceset="GND" device=""/>
 <part name="C13" library="SparkFun" deviceset="CAP" device="0603-CAP" value="0.1uF"/>
-<part name="R12" library="SparkFun" deviceset="RESISTOR" device="0603-RES"/>
-<part name="R13" library="SparkFun" deviceset="RESISTOR" device="0603-RES"/>
 <part name="S1" library="Testing" deviceset="SWITCH-MOMENTARY-2" device="SMD-ALT01" value="Reset"/>
 <part name="Q1" library="Testing" deviceset="RESONATOR" device="1:1" value="8/16/20MHz"/>
 <part name="JP1" library="SparkFun" deviceset="ARDUINO_SERIAL_PROGRAM" device="PTH" value="FTDI Basic"/>
 <part name="U$11" library="microbuilder" deviceset="3.3V" device=""/>
-<part name="U$13" library="microbuilder" deviceset="3.3V" device=""/>
-<part name="U$15" library="microbuilder" deviceset="3.3V" device=""/>
 <part name="U$16" library="microbuilder" deviceset="3.3V" device=""/>
 </parts>
@@
 <wire x1="0" y1="-220.98" x2="246.38" y2="-220.98" width="0.4064" layer="97" style="shortdash"/>
 <wire x1="0" y1="124.46" x2="0" y2="68.58" width="0.4064" layer="97" style="shortdash"/>
-<wire x1="0" y1="68.58" x2="2.54" y2="12.7" width="0.4064" layer="97" style="shortdash"/>
 <text x="40.64" y="104.14" size="1.778" layer="97">Place RN1 as close as possible
 to USB-Connector!</text>
@@
 <attribute name="VALUE" x="-68.961" y="-52.324" size="1.778" layer="96" rot="R90"/>
 </instance>
-<instance part="R12" gate="G$1" x="15.24" y="-58.42" rot="R90"/>
-<instance part="R13" gate="G$1" x="22.86" y="-60.96" rot="R90"/>
 <instance part="S1" gate="G$1" x="-63.5" y="-60.96" rot="R90"/>
 <instance part="Q1" gate="G$1" x="-40.64" y="-81.28" smashed="yes" rot="R270">
@@
 <instance part="JP1" gate="G$1" x="-20.32" y="-165.1"/>
 <instance part="U$11" gate="G$1" x="-40.64" y="-45.72"/>
-<instance part="U$13" gate="G$1" x="15.24" y="-45.72"/>
-<instance part="U$15" gate="G$1" x="22.86" y="-45.72"/>
 <instance part="U$16" gate="G$1" x="-63.5" y="-25.4"/>
 </instances>
@@
 </segment>
 <segment>
-<wire x1="15.24" y1="-53.34" x2="15.24" y2="-48.26" width="0.1524" layer="91"/>
-<pinref part="R12" gate="G$1" pin="2"/>
-<pinref part="U$13" gate="G$1" pin="3.3V"/>
-</segment>
-<segment>
-<wire x1="22.86" y1="-55.88" x2="22.86" y2="-48.26" width="0.1524" layer="91"/>
-<pinref part="R13" gate="G$1" pin="2"/>
-<pinref part="U$15" gate="G$1" pin="3.3V"/>
-</segment>
-<segment>
 <wire x1="-63.5" y1="-27.94" x2="-63.5" y2="-40.64" width="0.1524" layer="91"/>
 <pinref part="R8" gate="G$1" pin="2"/>
@@
 <label x="226.06" y="-76.2" size="1.778" layer="95"/>
 </segment>
-<segment>
-<wire x1="12.7" y1="-111.76" x2="12.7" y2="-114.3" width="0.1524" layer="91"/>
-<wire x1="7.62" y1="-111.76" x2="12.7" y2="-111.76" width="0.1524" layer="91"/>
-<pinref part="U4" gate="G$1" pin="PB5(SCK)"/>
-<pinref part="R11" gate="G$1" pin="1"/>
-</segment>
 </net>
 <net name="SWD_DIO" class="0">
@@
 <wire x1="213.36" y1="106.68" x2="213.36" y2="114.3" width="0.1524" layer="91"/>
 <label x="213.36" y="114.3" size="1.778" layer="95" rot="R180"/>
+</segment>
+<segment>
+<pinref part="U4" gate="G$1" pin="PC4(ADC4/SDA)"/>
+<wire x1="7.62" y1="-63.5" x2="17.78" y2="-63.5" width="0.1524" layer="91"/>
+<label x="17.78" y="-63.5" size="1.778" layer="95"/>
 </segment>
 </net>
@@
 <wire x1="218.44" y1="101.6" x2="218.44" y2="96.52" width="0.1524" layer="91"/>
 <label x="218.44" y="96.52" size="1.778" layer="95" rot="R180"/>
+</segment>
+<segment>
+<pinref part="U4" gate="G$1" pin="PC5(ADC5/SCL)"/>
+<wire x1="7.62" y1="-66.04" x2="27.94" y2="-66.04" width="0.1524" layer="91"/>
 </segment>
 </net>
@@
 </segment>
 </net>
-<net name="A5" class="0">
-<segment>
-<wire x1="7.62" y1="-66.04" x2="22.86" y2="-66.04" width="0.1524" layer="91"/>
-<pinref part="U4" gate="G$1" pin="PC5(ADC5/SCL)"/>
-<pinref part="R13" gate="G$1" pin="1"/>
-</segment>
-</net>
-<net name="A4" class="0">
-<segment>
-<wire x1="7.62" y1="-63.5" x2="15.24" y2="-63.5" width="0.1524" layer="91"/>
-<pinref part="U4" gate="G$1" pin="PC4(ADC4/SDA)"/>
-<pinref part="R12" gate="G$1" pin="1"/>
-</segment>
-</net>
 <net name="N$6" class="0">
 <segment>
@@
 </segment>
 </net>
+<net name="NONE" class="0">
+<segment>
+<wire x1="12.7" y1="-111.76" x2="12.7" y2="-114.3" width="0.1524" layer="91"/>
+<wire x1="7.62" y1="-111.76" x2="12.7" y2="-111.76" width="0.1524" layer="91"/>
+<pinref part="U4" gate="G$1" pin="PB5(SCK)"/>
+<pinref part="R11" gate="G$1" pin="1"/>
+</segment>
+</net>

Commit message: making mods to pins
Parts:
- added JP2, JP3, JP4, JP5, JP6, JP7: (no value), adafruit:PINHD-1X3
Connections:
- net GND: now also JP2.1, JP3.1, JP4.1, JP5.1, JP6.1, JP7.1
- net SCL: now also JP2.2, JP3.2, JP4.2, JP5.2, JP6.2, JP7.2
- net SDA: now also JP2.3, JP3.3, JP4.3, JP5.3, JP6.3, JP7.3
Changed lines of the file:
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@@
 <part name="U$11" library="microbuilder" deviceset="3.3V" device=""/>
 <part name="U$16" library="microbuilder" deviceset="3.3V" device=""/>
+<part name="JP2" library="adafruit" deviceset="PINHD-1X3" device=""/>
+<part name="GND15" library="supply1" deviceset="GND" device=""/>
+<part name="JP3" library="adafruit" deviceset="PINHD-1X3" device=""/>
+<part name="GND20" library="supply1" deviceset="GND" device=""/>
+<part name="JP4" library="adafruit" deviceset="PINHD-1X3" device=""/>
+<part name="GND21" library="supply1" deviceset="GND" device=""/>
+<part name="JP5" library="adafruit" deviceset="PINHD-1X3" device=""/>
+<part name="GND22" library="supply1" deviceset="GND" device=""/>
+<part name="JP6" library="adafruit" deviceset="PINHD-1X3" device=""/>
+<part name="GND23" library="supply1" deviceset="GND" device=""/>
+<part name="JP7" library="adafruit" deviceset="PINHD-1X3" device=""/>
+<part name="GND24" library="supply1" deviceset="GND" device=""/>
 </parts>
 <sheets>
@@
 <instance part="U$11" gate="G$1" x="-40.64" y="-45.72"/>
 <instance part="U$16" gate="G$1" x="-63.5" y="-25.4"/>
+<instance part="JP2" gate="A" x="-40.64" y="20.32" rot="R180"/>
+<instance part="GND15" gate="1" x="-30.48" y="17.78" rot="R90"/>
+<instance part="JP3" gate="A" x="-40.64" y="2.54" rot="R180"/>
+<instance part="GND20" gate="1" x="-30.48" y="0" rot="R90"/>
+<instance part="JP4" gate="A" x="-5.08" y="20.32" rot="R180"/>
+<instance part="GND21" gate="1" x="5.08" y="17.78" rot="R90"/>
+<instance part="JP5" gate="A" x="-5.08" y="2.54" rot="R180"/>
+<instance part="GND22" gate="1" x="5.08" y="0" rot="R90"/>
+<instance part="JP6" gate="A" x="-22.86" y="-15.24" rot="R180"/>
+<instance part="GND23" gate="1" x="-12.7" y="-17.78" rot="R90"/>
+<instance part="JP7" gate="A" x="-22.86" y="-33.02" rot="R180"/>
+<instance part="GND24" gate="1" x="-12.7" y="-35.56" rot="R90"/>
 </instances>
 <busses>
@@
 <pinref part="JP1" gate="G$1" pin="GND"/>
 <label x="-12.7" y="-157.48" size="1.27" layer="95" xref="yes"/>
+</segment>
+<segment>
+<pinref part="GND15" gate="1" pin="GND"/>
+<pinref part="JP2" gate="A" pin="1"/>
+<wire x1="-33.02" y1="17.78" x2="-38.1" y2="17.78" width="0.1524" layer="91"/>
+</segment>
+<segment>
+<pinref part="GND20" gate="1" pin="GND"/>
+<pinref part="JP3" gate="A" pin="1"/>
+<wire x1="-33.02" y1="0" x2="-38.1" y2="0" width="0.1524" layer="91"/>
+</segment>
+<segment>
+<pinref part="GND21" gate="1" pin="GND"/>
+<pinref part="JP4" gate="A" pin="1"/>
+<wire x1="2.54" y1="17.78" x2="-2.54" y2="17.78" width="0.1524" layer="91"/>
+</segment>
+<segment>
+<pinref part="GND22" gate="1" pin="GND"/>
+<pinref part="JP5" gate="A" pin="1"/>
+<wire x1="2.54" y1="0" x2="-2.54" y2="0" width="0.1524" layer="91"/>
+</segment>
+<segment>
+<pinref part="GND23" gate="1" pin="GND"/>
+<pinref part="JP6" gate="A" pin="1"/>
+<wire x1="-15.24" y1="-17.78" x2="-20.32" y2="-17.78" width="0.1524" layer="91"/>
+</segment>
+<segment>
+<pinref part="GND24" gate="1" pin="GND"/>
+<pinref part="JP7" gate="A" pin="1"/>
+<wire x1="-15.24" y1="-35.56" x2="-20.32" y2="-35.56" width="0.1524" layer="91"/>
 </segment>
 </net>
@@
 <label x="17.78" y="-63.5" size="1.778" layer="95"/>
 </segment>
+<segment>
+<pinref part="JP2" gate="A" pin="3"/>
+<wire x1="-38.1" y1="22.86" x2="-30.48" y2="22.86" width="0.1524" layer="91"/>
+<label x="-30.48" y="22.86" size="1.778" layer="95"/>
+</segment>
+<segment>
+<pinref part="JP3" gate="A" pin="3"/>
+<wire x1="-38.1" y1="5.08" x2="-30.48" y2="5.08" width="0.1524" layer="91"/>
+<label x="-30.48" y="5.08" size="1.778" layer="95"/>
+</segment>
+<segment>
+<pinref part="JP4" gate="A" pin="3"/>
+<wire x1="-2.54" y1="22.86" x2="5.08" y2="22.86" width="0.1524" layer="91"/>
+<label x="5.08" y="22.86" size="1.778" layer="95"/>
+</segment>
+<segment>
+<pinref part="JP5" gate="A" pin="3"/>
+<wire x1="-2.54" y1="5.08" x2="5.08" y2="5.08" width="0.1524" layer="91"/>
+<label x="5.08" y="5.08" size="1.778" layer="95"/>
+</segment>
+<segment>
+<pinref part="JP6" gate="A" pin="3"/>
+<wire x1="-20.32" y1="-12.7" x2="-12.7" y2="-12.7" width="0.1524" layer="91"/>
+<label x="-12.7" y="-12.7" size="1.778" layer="95"/>
+</segment>
+<segment>
+<pinref part="JP7" gate="A" pin="3"/>
+<wire x1="-20.32" y1="-30.48" x2="-12.7" y2="-30.48" width="0.1524" layer="91"/>
+<label x="-12.7" y="-30.48" size="1.778" layer="95"/>
+</segment>
 </net>
 <net name="SCL" class="0">
@@
 <wire x1="7.62" y1="-66.04" x2="27.94" y2="-66.04" width="0.1524" layer="91"/>
 </segment>
-</net>
+<segment>
+<wire x1="-38.1" y1="20.32" x2="-45.72" y2="20.32" width="0.1524" layer="91"/>
+<label x="-50.8" y="20.32" size="1.778" layer="95"/>
+<pinref part="JP2" gate="A" pin="2"/>
+</segment>
+<segment>
+<wire x1="-38.1" y1="2.54" x2="-45.72" y2="2.54" width="0.1524" layer="91"/>
+<label x="-50.8" y="2.54" size="1.778" layer="95"/>
+<pinref part="JP3" gate="A" pin="2"/>
+</segment>
+<segment>
+<wire x1="-2.54" y1="20.32" x2="-10.16" y2="20.32" width="0.1524" layer="91"/>
+<label x="-15.24" y="20.32" size="1.778" layer="95"/>
+<pinref part="JP4" gate="A" pin="2"/>
+</segment>
+<segment>
+<wire x1="-2.54" y1="2.54" x2="-10.16" y2="2.54" width="0.1524" layer="91"/>
+<label x="-15.24" y="2.54" size="1.778" layer="95"/>
+<pinref part="JP5" gate="A" pin="2"/>
+</segment>
+<segment>
+<wire x1="-20.32" y1="-15.24" x2="-27.94" y2="-15.24" width="0.1524" layer="91"/>
+<label x="-33.02" y="-15.24" size="1.778" layer="95"/>
+<pinref part="JP6" gate="A" pin="2"/>
+</segment>
+<segment>
+<wire x1="-20.32" y1="-33.02" x2="-27.94" y2="-33.02" width="0.1524" layer="91"/>
+<label x="-33.02" y="-33.02" size="1.778" layer="95"/>
+<pinref part="JP7" gate="A" pin="2"/>
+</segment>
+</net>

Commit message: wiring attempting
Parts:
- added JP10, JP11, JP8, JP9: (no value), adafruit:PINHD-1X3
Connections:
- new net N$11: JP10.3, U4.PD2(INT0)
- new net N$13: JP9.3, U4.PD3(INT1)
- new net N$14: JP8.3, U4.PD4(XCK/T0)
- new net N$16: JP11.3, U4.PD5(T1)
- net GND: now also JP10.1, JP11.1, JP8.1, JP9.1
Changed lines of the file:
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@@
 <part name="JP7" library="adafruit" deviceset="PINHD-1X3" device=""/>
 <part name="GND24" library="supply1" deviceset="GND" device=""/>
+<part name="JP8" library="adafruit" deviceset="PINHD-1X3" device=""/>
+<part name="GND25" library="supply1" deviceset="GND" device=""/>
+<part name="JP9" library="adafruit" deviceset="PINHD-1X3" device=""/>
+<part name="GND26" library="supply1" deviceset="GND" device=""/>
+<part name="JP10" library="adafruit" deviceset="PINHD-1X3" device=""/>
+<part name="GND27" library="supply1" deviceset="GND" device=""/>
+<part name="JP11" library="adafruit" deviceset="PINHD-1X3" device=""/>
+<part name="GND28" library="supply1" deviceset="GND" device=""/>
 </parts>
 <sheets>
@@
 <instance part="JP7" gate="A" x="-22.86" y="-33.02" rot="R180"/>
 <instance part="GND24" gate="1" x="-12.7" y="-35.56" rot="R90"/>
+<instance part="JP8" gate="A" x="27.94" y="-20.32"/>
+<instance part="GND25" gate="1" x="17.78" y="-17.78" rot="R270"/>
+<instance part="JP9" gate="A" x="27.94" y="-35.56"/>
+<instance part="GND26" gate="1" x="17.78" y="-33.02" rot="R270"/>
+<instance part="JP10" gate="A" x="27.94" y="-50.8"/>
+<instance part="GND27" gate="1" x="17.78" y="-48.26" rot="R270"/>
+<instance part="JP11" gate="A" x="27.94" y="-2.54"/>
+<instance part="GND28" gate="1" x="17.78" y="0" rot="R270"/>
 </instances>
 <busses>
@@
 <pinref part="JP7" gate="A" pin="1"/>
 <wire x1="-15.24" y1="-35.56" x2="-20.32" y2="-35.56" width="0.1524" layer="91"/>
+</segment>
+<segment>
+<pinref part="JP8" gate="A" pin="1"/>
+<pinref part="GND25" gate="1" pin="GND"/>
+<wire x1="25.4" y1="-17.78" x2="20.32" y2="-17.78" width="0.1524" layer="91"/>
+</segment>
+<segment>
+<pinref part="JP9" gate="A" pin="1"/>
+<pinref part="GND26" gate="1" pin="GND"/>
+<wire x1="25.4" y1="-33.02" x2="20.32" y2="-33.02" width="0.1524" layer="91"/>
+</segment>
+<segment>
+<pinref part="JP10" gate="A" pin="1"/>
+<pinref part="GND27" gate="1" pin="GND"/>
+<wire x1="25.4" y1="-48.26" x2="20.32" y2="-48.26" width="0.1524" layer="91"/>
+</segment>
+<segment>
+<pinref part="JP11" gate="A" pin="1"/>
+<pinref part="GND28" gate="1" pin="GND"/>
+<wire x1="25.4" y1="0" x2="20.32" y2="0" width="0.1524" layer="91"/>
 </segment>
 </net>
@@
 </segment>
 </net>
+<net name="N$11" class="0">
+<segment>
+<pinref part="JP10" gate="A" pin="3"/>
+<wire x1="25.4" y1="-53.34" x2="30.48" y2="-53.34" width="0.1524" layer="91"/>
+<wire x1="30.48" y1="-53.34" x2="30.48" y2="-81.28" width="0.1524" layer="91"/>
+<pinref part="U4" gate="G$1" pin="PD2(INT0)"/>
+<wire x1="30.48" y1="-81.28" x2="7.62" y2="-81.28" width="0.1524" layer="91"/>
+</segment>
+</net>
+<net name="N$13" class="0">
+<segment>
+<pinref part="JP9" gate="A" pin="3"/>
+<wire x1="25.4" y1="-38.1" x2="33.02" y2="-38.1" width="0.1524" layer="91"/>
+<wire x1="33.02" y1="-38.1" x2="33.02" y2="-83.82" width="0.1524" layer="91"/>
+<pinref part="U4" gate="G$1" pin="PD3(INT1)"/>
+<wire x1="33.02" y1="-83.82" x2="7.62" y2="-83.82" width="0.1524" layer="91"/>
+</segment>
+</net>
+<net name="N$14" class="0">
+<segment>
+<pinref part="JP8" gate="A" pin="3"/>
+<wire x1="25.4" y1="-22.86" x2="35.56" y2="-22.86" width="0.1524" layer="91"/>
+<wire x1="35.56" y1="-22.86" x2="35.56" y2="-86.36" width="0.1524" layer="91"/>
+<pinref part="U4" gate="G$1" pin="PD4(XCK/T0)"/>
+<wire x1="35.56" y1="-86.36" x2="7.62" y2="-86.36" width="0.1524" layer="91"/>
+</segment>
+</net>
+<net name="N$16" class="0">
+<segment>
+<pinref part="JP11" gate="A" pin="3"/>
+<wire x1="25.4" y1="-5.08" x2="38.1" y2="-5.08" width="0.1524" layer="91"/>
+<wire x1="38.1" y1="-5.08" x2="38.1" y2="-88.9" width="0.1524" layer="91"/>
+<pinref part="U4" gate="G$1" pin="PD5(T1)"/>
+<wire x1="38.1" y1="-88.9" x2="7.62" y2="-88.9" width="0.1524" layer="91"/>
+</segment>
+</net>
