File: Flight-Controller-PCB1/flight-controller.brd (EAGLE design)
At the start: 100 x 25.4 mm, 37 parts, among them J1 1981584-1, U1 MK20DX256VLH7, U2 TPS61200, U3 MINI54TAN, Y1 32.768KHz, Y2 16Mhz/8pF

Commit message: update
Parts:
- moved RN1 3.81 mm to (10.2, 12.7)
Routing:
- net USB_CON_P: track 1.75 -> 5.55 mm
- net USB_CON_N: track 1.66 -> 5.44 mm
Other:
- board size 100 x 25.4 mm -> 100 x 27.9 mm
Changed lines of the file:
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@@
 <board>
 <plain>
-<wire x1="0" y1="0" x2="100" y2="0" width="0" layer="20"/>
-<wire x1="100" y1="0" x2="100" y2="25.39" width="0" layer="20"/>
-<wire x1="100" y1="25.39" x2="0" y2="25.39" width="0" layer="20"/>
-<wire x1="0" y1="25.39" x2="0" y2="0" width="0" layer="20"/>
+<wire x1="0" y1="-1.27" x2="100" y2="-1.27" width="0" layer="20"/>
+<wire x1="100" y1="-1.27" x2="100" y2="26.66" width="0" layer="20"/>
+<wire x1="100" y1="26.66" x2="0" y2="26.66" width="0" layer="20"/>
+<wire x1="0" y1="26.66" x2="0" y2="-1.27" width="0" layer="20"/>
 </plain>
 <attributes>
@@
 <attribute name="MF" value="Panasonic" x="3.81" y="1.27" size="1.778" layer="27" display="off"/>
 </element>
-<element name="RN1" library="resistor-dil" package="EXB34V" value="33" x="6.35" y="12.7" rot="R270">
-<attribute name="MPN" value="EXB-34V330JV" x="6.35" y="12.7" size="1.778" layer="27" rot="R270" display="off"/>
-<attribute name="OC_NEWARK" value="unknown" x="6.35" y="12.7" size="1.778" layer="27" rot="R270" display="off"/>
-<attribute name="MF" value="Panasonic" x="6.35" y="12.7" size="1.778" layer="27" rot="R270" display="off"/>
-<attribute name="OC_FARNELL" value="unknown" x="6.35" y="12.7" size="1.778" layer="27" rot="R270" display="off"/>
+<element name="RN1" library="resistor-dil" package="EXB34V" value="33" x="10.16" y="12.7" rot="R270">
+<attribute name="MPN" value="EXB-34V330JV" x="10.16" y="12.7" size="1.778" layer="27" rot="R270" display="off"/>
+<attribute name="OC_NEWARK" value="unknown" x="10.16" y="12.7" size="1.778" layer="27" rot="R270" display="off"/>
+<attribute name="MF" value="Panasonic" x="10.16" y="12.7" size="1.778" layer="27" rot="R270" display="off"/>
+<attribute name="OC_FARNELL" value="unknown" x="10.16" y="12.7" size="1.778" layer="27" rot="R270" display="off"/>
 </element>
 <element name="U1" library="appfruits" package="MK20DX256VLH7" value="MK20DX256VLH7" x="53.34" y="13.97" rot="R270">
@@
 <contactref element="U1" pad="5"/>
 <contactref element="RN1" pad="3"/>
-<wire x1="7.05" y1="12.2" x2="55.09" y2="19.67" width="0" layer="19" extent="1-1"/>
+<wire x1="10.86" y1="12.2" x2="55.09" y2="19.67" width="0" layer="19" extent="1-1"/>
 </signal>
 <signal name="USB_D_N" class="1">
 <contactref element="RN1" pad="4"/>
 <contactref element="U1" pad="6"/>
-<wire x1="7.05" y1="13.2" x2="54.59" y2="19.67" width="0" layer="19" extent="1-1"/>
+<wire x1="10.86" y1="13.2" x2="54.59" y2="19.67" width="0" layer="19" extent="1-1"/>
 </signal>
 <signal name="ID">
@@
 <contactref element="RN1" pad="1"/>
 <wire x1="4.1148" y1="13.2588" x2="5.6007" y2="13.2588" width="0.254" layer="1"/>
-<wire x1="5.6007" y1="13.2588" x2="5.65" y2="13.2" width="0.254" layer="1"/>
+<wire x1="5.6007" y1="13.2588" x2="9.46" y2="13.2" width="0.254" layer="1"/>
 <wire x1="4.1148" y1="13.2588" x2="4.1" y2="13.35" width="0.254" layer="1"/>
 </signal>
@@
 <wire x1="5.1435" y1="12.6873" x2="5.6007" y2="12.2301" width="0.254" layer="1"/>
 <wire x1="4.1148" y1="12.6873" x2="5.1435" y2="12.6873" width="0.254" layer="1"/>
-<wire x1="5.6007" y1="12.2301" x2="5.65" y2="12.2" width="0.254" layer="1"/>
+<wire x1="5.6007" y1="12.2301" x2="9.46" y2="12.2" width="0.254" layer="1"/>
 <wire x1="4.1148" y1="12.6873" x2="4.1" y2="12.7" width="0.254" layer="1"/>
 </signal>

Commit message: started manually routing
Parts:
- moved R2 2.54 mm to (22.9, 22.9)
- moved R3 2.54 mm to (20.3, 22.9)
- moved U2 1.27 mm to (14.0, 22.9), turned to 90 degrees
- moved L1 1.27 mm to (15.2, 16.5)
- moved R6 1.27 mm to (2.54, 24.1)
Routing:
- net GND: track 161.3 -> 5.15 mm, vias 5 -> 0
- net 3.3V: track 161.0 -> 21.1 mm, vias 7 -> 2
- net ID: track 72.7 -> 0.00 mm, vias 3 -> 0
- net VCC: track 54.1 -> 4.73 mm, vias 5 -> 0
- net RESET_B: track 47.2 -> 0.00 mm, vias 2 -> 0
- net VDDA: track 40.5 -> 0.00 mm, vias 3 -> 0
- net PGND: track 32.3 -> 0.00 mm, vias 5 -> 0
- net UVLO: track 28.0 -> 0.00 mm, vias 2 -> 0
- net VREFL: track 23.2 -> 0.00 mm
- net N$19: track 22.5 -> 0.00 mm
- net SWD_CLK: track 21.2 -> 0.00 mm, vias 2 -> 0
- net SWD_DIO: track 20.6 -> 0.00 mm
- net VAUX: track 15.1 -> 0.00 mm, vias 2 -> 0
- net N$22: track 12.0 -> 0.00 mm, vias 2 -> 0
- net VREF_OUT: track 11.3 -> 0.00 mm
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
Commit message: still routing
Routing:
- net UVLO: track 0.00 -> 32.3 mm, vias 0 -> 3
Changed lines of the file:
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@@
 <contactref element="R3" pad="1"/>
 <contactref element="R4" pad="2"/>
-<wire x1="12.495" y1="23.36" x2="20.32" y2="23.71" width="0" layer="19" extent="1-1"/>
-<wire x1="10.58" y1="1.27" x2="12.495" y2="23.36" width="0" layer="19" extent="1-1"/>
 <wire x1="8.47" y1="1.27" x2="10.58" y2="1.27" width="0" layer="19" extent="1-1"/>
+<wire x1="20.32" y1="23.71" x2="20.32" y2="25.4" width="0.254" layer="1"/>
+<wire x1="20.32" y1="25.4" x2="19.812" y2="25.908" width="0.254" layer="1"/>
+<wire x1="19.812" y1="25.908" x2="19.05" y2="25.908" width="0.254" layer="1"/>
+<wire x1="19.05" y1="25.908" x2="18.542" y2="25.4" width="0.254" layer="1"/>
+<wire x1="18.542" y1="25.4" x2="18.542" y2="20.828" width="0.254" layer="1"/>
+<wire x1="18.542" y1="20.828" x2="17.526" y2="19.812" width="0.254" layer="1"/>
+<wire x1="17.526" y1="19.812" x2="13.462" y2="19.812" width="0.254" layer="1"/>
+<via x="13.462" y="19.812" extent="1-16" drill="0.5"/>
+<wire x1="13.462" y1="19.812" x2="10.668" y2="19.812" width="0.254" layer="16"/>
+<wire x1="10.668" y1="19.812" x2="10.414" y2="20.066" width="0.254" layer="16"/>
+<wire x1="12.495" y1="23.36" x2="11.676" y2="23.36" width="0.254" layer="1"/>
+<wire x1="11.676" y1="23.36" x2="10.414" y2="22.098" width="0.254" layer="1"/>
+<wire x1="10.414" y1="22.098" x2="10.414" y2="20.066" width="0.254" layer="1"/>
+<via x="10.414" y="20.066" extent="1-16" drill="0.5"/>
+<wire x1="10.414" y1="20.066" x2="10.414" y2="17.78" width="0.254" layer="16"/>
+<wire x1="10.414" y1="17.78" x2="8.89" y2="16.256" width="0.254" layer="16"/>
+<wire x1="8.89" y1="16.256" x2="8.89" y2="11.176" width="0.254" layer="16"/>
+<via x="8.89" y="11.176" extent="1-16" drill="0.5"/>
+<wire x1="8.89" y1="11.176" x2="8.89" y2="10.16" width="0.254" layer="1"/>
+<wire x1="8.89" y1="10.16" x2="8.47" y2="1.27" width="0" layer="19" extent="1-16"/>
 </signal>
 <signal name="FB">

Commit message: continuing manual routing
Routing:
- net GND: track 5.15 -> 58.7 mm, vias 0 -> 4
- net VCC: track 4.73 -> 53.4 mm, vias 0 -> 3
- net PGND: track 0.00 -> 48.5 mm, vias 0 -> 6
- net ID: track 0.00 -> 44.4 mm, vias 0 -> 2
- net 3.3V: track 21.1 -> 59.0 mm
- net VAUX: track 0.00 -> 18.9 mm, vias 0 -> 2
- net UVLO: track 32.3 -> 43.5 mm
- net N$2: track 0.00 -> 10.8 mm
- net USB_CON_P: track 0.00 -> 5.57 mm
- net USB_CON_N: track 0.00 -> 5.42 mm
- net N$1: track 0.00 -> 1.85 mm
- net USB_SHIELD: track 16.4 -> 17.3 mm

Commit message: nearly finished routing
Routing:
- net GND: track 58.7 -> 198.5 mm, vias 4 -> 12
- net 3.3V: track 59.0 -> 154.6 mm, vias 2 -> 5
- net SWD_DIO: track 0.00 -> 40.4 mm, vias 0 -> 2
- net VREFH: track 0.00 -> 35.6 mm, vias 0 -> 2
- net RESET_B: track 0.00 -> 28.0 mm, vias 0 -> 2
- net VDDA: track 0.00 -> 27.6 mm, vias 0 -> 2
- net SWD_CLK: track 0.00 -> 26.4 mm, vias 0 -> 4
- net N$15: track 0.00 -> 26.0 mm, vias 0 -> 4
- net VREFL: track 0.00 -> 24.4 mm
- net N$19: track 0.00 -> 22.5 mm, vias 0 -> 2
- net ID: track 44.4 -> 66.0 mm, vias 2 -> 4
- net PS: track 0.00 -> 20.0 mm, vias 0 -> 4
- net N$12: track 0.00 -> 14.2 mm
- net VREF_OUT: track 0.00 -> 12.4 mm, vias 0 -> 2
- net N$27: track 0.00 -> 10.7 mm
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Other:
- board size 100 x 27.9 mm -> 79.9 x 27.9 mm

Commit message: finished traces
Routing:
- net USB_D_N: track 0.00 -> 57.3 mm, vias 0 -> 2
- net USB_D_P: track 0.00 -> 51.3 mm, vias 0 -> 4
Changed lines of the file:
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@@
 <contactref element="U1" pad="5"/>
 <contactref element="RN1" pad="3"/>
-<wire x1="10.86" y1="12.2" x2="55.09" y2="19.67" width="0" layer="19" extent="1-1"/>
+<wire x1="32.258" y1="15.748" x2="33.782" y2="17.272" width="0.254" layer="1"/>
+<via x="33.782" y="17.272" extent="1-16" drill="0.6096"/>
+<wire x1="33.782" y1="17.272" x2="44.704" y2="17.272" width="0.254" layer="16"/>
+<wire x1="44.704" y1="17.272" x2="48.514" y2="21.082" width="0.254" layer="16"/>
+<wire x1="48.514" y1="21.082" x2="53.594" y2="21.082" width="0.254" layer="16"/>
+<wire x1="53.594" y1="21.082" x2="54.61" y2="22.098" width="0.254" layer="16"/>
+<via x="54.61" y="22.098" extent="1-16" drill="0.5"/>
+<wire x1="54.61" y1="22.098" x2="54.864" y2="22.098" width="0.254" layer="1"/>
+<wire x1="54.864" y1="22.098" x2="55.372" y2="21.59" width="0.254" layer="1"/>
+<wire x1="55.372" y1="21.59" x2="55.372" y2="21.082" width="0.254" layer="1"/>
+<wire x1="55.372" y1="21.082" x2="55.118" y2="20.828" width="0.254" layer="1"/>
+<wire x1="55.118" y1="20.828" x2="55.118" y2="19.698" width="0.254" layer="1"/>
+<wire x1="55.118" y1="19.698" x2="55.09" y2="19.67" width="0.254" layer="1"/>
+<wire x1="10.86" y1="12.2" x2="18.534" y2="12.2" width="0.254" layer="1"/>
+<wire x1="18.534" y1="12.2" x2="19.05" y2="11.684" width="0.254" layer="1"/>
+<wire x1="19.05" y1="11.684" x2="20.32" y2="11.684" width="0.254" layer="1"/>
+<via x="20.32" y="11.684" extent="1-16" drill="0.6096"/>
+<wire x1="20.32" y1="11.684" x2="22.606" y2="11.684" width="0.254" layer="16"/>
+<wire x1="22.606" y1="11.684" x2="26.67" y2="15.748" width="0.254" layer="16"/>
+<wire x1="26.67" y1="15.748" x2="30.48" y2="15.748" width="0.254" layer="16"/>
+<via x="30.48" y="15.748" extent="1-16" drill="0.5"/>
+<wire x1="30.48" y1="15.748" x2="32.258" y2="15.748" width="0.254" layer="1"/>
 </signal>
 <signal name="USB_D_N" class="1">
 <contactref element="RN1" pad="4"/>
 <contactref element="U1" pad="6"/>
-<wire x1="10.86" y1="13.2" x2="54.59" y2="19.67" width="0" layer="19" extent="1-1"/>
+<wire x1="10.86" y1="13.2" x2="20.312" y2="13.2" width="0.254" layer="1"/>
+<wire x1="20.312" y1="13.2" x2="20.32" y2="13.208" width="0.254" layer="1"/>
+<via x="20.32" y="13.208" extent="1-16" drill="0.6096"/>
+<wire x1="20.32" y1="13.208" x2="22.352" y2="13.208" width="0.254" layer="16"/>
+<wire x1="22.352" y1="13.208" x2="23.622" y2="14.478" width="0.254" layer="16"/>
+<wire x1="23.622" y1="14.478" x2="23.622" y2="24.13" width="0.254" layer="16"/>
+<wire x1="23.622" y1="24.13" x2="24.638" y2="25.146" width="0.254" layer="16"/>
+<wire x1="24.638" y1="25.146" x2="50.292" y2="25.146" width="0.254" layer="16"/>
+<wire x1="50.292" y1="25.146" x2="53.34" y2="22.098" width="0.254" layer="16"/>
+<via x="53.34" y="22.098" extent="1-16" drill="0.6096"/>
+<wire x1="53.34" y1="22.098" x2="54.59" y2="20.848" width="0.254" layer="1"/>
+<wire x1="54.59" y1="20.848" x2="54.59" y2="19.67" width="0.254" layer="1"/>
 </signal>
 <signal name="ID">

Commit message: finished setting up my portion
Parts:
- added C6, C8: 0.1uF, appfruits:0603-CAP
- added C7: 10nF, appfruits:0603-CAP
- added C9: 2.2nF, appfruits:0603-CAP
- added R1, R5: 10K, appfruits:0603-RES
- added SJ1: (no value), jumper:SJ_2
- added U$1: MPU-9150.QFN, invensense:QFN.24.4X4
Connections:
- new net N$3: C9.1, U$1.20
- new net N$4: C8.1, U$1.10
- new net N$5: SJ1.2, U$1.9
- net 3.3V: now also C6.1, C7.1, R1.1, R5.1, SJ1.1, U$1.13, U$1.3, U$1.8
- net GND: now also C6.2, C7.2, C8.2, C9.2, SJ1.3, U$1.15, U$1.17, U$1.18
- net SCL: now also R5.2, U$1.23
- net SDA: now also R1.2, U$1.24
Routing:
- net PS: track 20.0 -> 21.0 mm
Changed lines of the file:
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@@
 <attribute name="MF" value="ECS" x="50.8" y="2.54" size="1.778" layer="27" rot="R180" display="off"/>
+</element>
+<element name="U$1" library="invensense" package="QFN.24.4X4" value="MPU-9150.QFN" x="68.58" y="21.844" rot="R180"/>
+<element name="C6" library="appfruits" package="0603-CAP" value="0.1uF" x="66.548" y="8.128">
+<attribute name="MPN" value="C0603C104J3RACTU" x="66.548" y="8.128" size="1.778" layer="27" display="off"/>
+<attribute name="MF" value="Kemet" x="66.548" y="8.128" size="1.778" layer="27" display="off"/>
+</element>
+<element name="C7" library="appfruits" package="0603-CAP" value="10nF" x="66.548" y="4.826">
+<attribute name="MPN" value="C0603C104J3RACTU" x="66.548" y="4.826" size="1.778" layer="27" display="off"/>
+<attribute name="MF" value="Kemet" x="66.548" y="4.826" size="1.778" layer="27" display="off"/>
+</element>
+<element name="C8" library="appfruits" package="0603-CAP" value="0.1uF" x="66.548" y="11.938">
+<attribute name="MPN" value="C0603C104J3RACTU" x="66.548" y="11.938" size="1.778" layer="27" display="off"/>
+<attribute name="MF" value="Kemet" x="66.548" y="11.938" size="1.778" layer="27" display="off"/>
+</element>
+<element name="C9" library="appfruits" package="0603-CAP" value="2.2nF" x="66.548" y="15.24">
+<attribute name="MPN" value="C0603C104J3RACTU" x="66.548" y="15.24" size="1.778" layer="27" display="off"/>
+<attribute name="MF" value="Kemet" x="66.548" y="15.24" size="1.778" layer="27" display="off"/>
+</element>
+<element name="SJ1" library="jumper" package="SJ_2" value="" x="60.452" y="24.638"/>
+<element name="R1" library="appfruits" package="0603-RES" value="10K" x="71.374" y="15.24" rot="R180">
+<attribute name="MPN" value="ERJ-3GEYJ103V" x="71.374" y="15.24" size="1.778" layer="27" rot="R180" display="off"/>
+<attribute name="MF" value="Panasonic" x="71.374" y="15.24" size="1.778" layer="27" rot="R180" display="off"/>
+</element>
+<element name="R5" library="appfruits" package="0603-RES" value="10K" x="71.374" y="11.938" rot="R180">
+<attribute name="MPN" value="ERJ-3GEYJ103V" x="71.374" y="11.938" size="1.778" layer="27" rot="R180" display="off"/>
+<attribute name="MF" value="Panasonic" x="71.374" y="11.938" size="1.778" layer="27" rot="R180" display="off"/>
 </element>
 </elements>
@@
 <wire x1="49.022" y1="10.668" x2="47.692" y2="10.668" width="0.254" layer="1"/>
 <wire x1="47.692" y1="10.668" x2="47.64" y2="10.72" width="0.254" layer="1"/>
+<contactref element="C6" pad="2"/>
+<contactref element="C7" pad="2"/>
+<contactref element="C9" pad="2"/>
+<contactref element="C8" pad="2"/>
+<contactref element="U$1" pad="15"/>
+<contactref element="U$1" pad="18"/>
+<contactref element="U$1" pad="17"/>
+<contactref element="SJ1" pad="3"/>
+<wire x1="66.605" y1="21.094" x2="66.605" y2="22.094" width="0" layer="19" extent="1-1"/>
+<wire x1="66.605" y1="20.594" x2="66.605" y2="21.094" width="0" layer="19" extent="1-1"/>
+<wire x1="62.992" y1="20.574" x2="66.605" y2="21.094" width="0" layer="19" extent="1-16"/>
+<wire x1="61.976" y1="24.638" x2="61.722" y2="21.844" width="0" layer="19" extent="1-16"/>
+<wire x1="67.398" y1="4.826" x2="62.992" y2="2.54" width="0" layer="19" extent="1-16"/>
+<wire x1="67.398" y1="8.128" x2="67.398" y2="4.826" width="0" layer="19" extent="1-1"/>
+<wire x1="67.398" y1="11.938" x2="67.398" y2="8.128" width="0" layer="19" extent="1-1"/>
+<wire x1="67.398" y1="15.24" x2="67.398" y2="11.938" width="0" layer="19" extent="1-1"/>
 </signal>
 <signal name="N$2">
@@
 <wire x1="5.842" y1="25.146" x2="16.764" y2="25.146" width="0.254" layer="16"/>
 <wire x1="16.764" y1="25.146" x2="17.526" y2="24.384" width="0.254" layer="16"/>
-<wire x1="17.526" y1="24.384" x2="17.526" y2="22.86" width="0.254" layer="16"/>
-<wire x1="17.526" y1="22.86" x2="17.018" y2="22.352" width="0.254" layer="16"/>
+<wire x1="17.526" y1="24.384" x2="17.526" y2="23.368" width="0.254" layer="16"/>
+<wire x1="17.526" y1="23.368" x2="17.018" y2="22.352" width="0.254" layer="16"/>
 <via x="17.018" y="22.352" extent="1-16" drill="0.5"/>
 <wire x1="17.018" y1="22.352" x2="15.453" y2="22.352" width="0.254" layer="1"/>
@@
 <wire x1="55.88" y1="10.668" x2="51.816" y2="10.668" width="0.254" layer="1"/>
 <wire x1="51.816" y1="10.668" x2="50.8" y2="11.684" width="0.254" layer="1"/>
+<contactref element="C6" pad="1"/>
+<contactref element="C7" pad="1"/>
+<contactref element="U$1" pad="13"/>
+<contactref element="U$1" pad="3"/>
+<contactref element="U$1" pad="8"/>
+<contactref element="R5" pad="1"/>
+<contactref element="R1" pad="1"/>
+<contactref element="SJ1" pad="1"/>
+<wire x1="70.555" y1="21.594" x2="69.33" y2="23.819" width="0" layer="19" extent="1-1"/>
+<wire x1="66.605" y1="23.094" x2="69.33" y2="23.819" width="0" layer="19" extent="1-1"/>
+<wire x1="58.928" y1="24.638" x2="66.605" y2="23.094" width="0" layer="19" extent="1-1"/>
+<wire x1="56.09" y1="19.67" x2="58.928" y2="24.638" width="0" layer="19" extent="1-1"/>
+<wire x1="72.224" y1="15.24" x2="70.555" y2="21.594" width="0" layer="19" extent="1-1"/>
+<wire x1="72.224" y1="11.938" x2="72.224" y2="15.24" width="0" layer="19" extent="1-1"/>
+<wire x1="65.698" y1="8.128" x2="72.224" y2="11.938" width="0" layer="19" extent="1-1"/>
+<wire x1="65.698" y1="4.826" x2="65.698" y2="8.128" width="0" layer="19" extent="1-1"/>
 </signal>
 <signal name="PS">
@@
 <contactref element="R2" pad="2"/>
 <wire x1="12.495" y1="22.86" x2="11.938" y2="22.86" width="0.254" layer="1"/>
-<wire x1="11.938" y1="22.86" x2="11.43" y2="22.352" width="0.254" layer="1"/>
-<wire x1="11.43" y1="22.352" x2="11.43" y2="21.844" width="0.254" layer="1"/>
-<via x="11.43" y="21.844" extent="1-16" drill="0.6096"/>
-<wire x1="11.43" y1="21.844" x2="11.43" y2="22.86" width="0.254" layer="16"/>
-<wire x1="11.43" y1="22.86" x2="10.16" y2="24.13" width="0.254" layer="16"/>
+<wire x1="11.938" y1="22.86" x2="11.176" y2="22.352" width="0.254" layer="1"/>
+<wire x1="11.176" y1="22.352" x2="11.176" y2="21.336" width="0.254" layer="1"/>
+<via x="11.176" y="21.336" extent="1-16" drill="0.6096"/>
+<wire x1="11.176" y1="21.336" x2="11.176" y2="22.606" width="0.254" layer="16"/>
+<wire x1="11.176" y1="22.606" x2="10.16" y2="24.13" width="0.254" layer="16"/>
 <via x="10.16" y="24.13" extent="1-16" drill="0.6096"/>
 <wire x1="10.16" y1="24.13" x2="10.16" y2="24.892" width="0.254" layer="1"/>
@@
 <contactref element="U3" pad="32"/>
 <contactref element="U1" pad="22"/>
-<wire x1="47.64" y1="15.22" x2="45.7" y2="15.22" width="0.254" layer="1"/>
-<wire x1="45.7" y1="15.22" x2="44.196" y2="13.716" width="0.254" layer="1"/>
-<wire x1="44.196" y1="13.716" x2="44.196" y2="11.684" width="0.254" layer="1"/>
+<wire x1="47.64" y1="15.22" x2="46.228" y2="15.22" width="0.254" layer="1"/>
+<wire x1="46.228" y1="15.22" x2="45.7" y2="15.22" width="0.254" layer="1"/>
+<wire x1="44.196" y1="14.224" x2="44.196" y2="11.684" width="0.254" layer="1"/>
 <wire x1="44.196" y1="11.684" x2="42.164" y2="9.652" width="0.254" layer="1"/>
 <via x="42.164" y="9.652" extent="1-16" drill="0.5"/>
@@
 <wire x1="32.512" y1="0" x2="32.512" y2="1.838" width="0.254" layer="1"/>
 <wire x1="32.512" y1="1.838" x2="32.5" y2="1.85" width="0.254" layer="1"/>
+<wire x1="44.196" y1="14.224" x2="45.192" y2="15.22" width="0.254" layer="1"/>
+<wire x1="45.192" y1="15.22" x2="45.7" y2="15.22" width="0.254" layer="1"/>
 </signal>
 <signal name="N$15">
@@
 <signal name="SDA">
 <contactref element="U1" pad="38"/>
+<contactref element="R1" pad="2"/>
+<contactref element="U$1" pad="24"/>
+<wire x1="69.83" y1="19.869" x2="70.524" y2="15.24" width="0" layer="19" extent="1-1"/>
+<wire x1="52.09" y1="8.27" x2="69.83" y2="19.869" width="0" layer="19" extent="1-1"/>
 </signal>
 <signal name="SCL">
 <contactref element="U1" pad="37"/>
+<contactref element="R5" pad="2"/>
+<contactref element="U$1" pad="23"/>
+<wire x1="70.524" y1="11.938" x2="69.33" y2="19.869" width="0" layer="19" extent="1-1"/>
+<wire x1="51.59" y1="8.27" x2="70.524" y2="11.938" width="0" layer="19" extent="1-1"/>
 </signal>
 <signal name="N$19">
@@
 <wire x1="6.858" y1="9.906" x2="8.724" y2="9.906" width="0.3048" layer="1"/>
 <wire x1="8.724" y1="9.906" x2="8.89" y2="9.74" width="0.3048" layer="1"/>
-<wire x1="11.01" y1="5.08" x2="12.192" y2="5.08" width="0.3048" layer="1"/>
-<via x="12.192" y="5.08" extent="1-16" drill="0.5"/>
-<wire x1="12.192" y1="5.08" x2="12.192" y2="7.874" width="0.3048" layer="16"/>
-<via x="12.192" y="7.874" extent="1-16" drill="0.5"/>
-<wire x1="12.192" y1="7.874" x2="10.326" y2="9.74" width="0.3048" layer="1"/>
+<wire x1="11.01" y1="5.08" x2="12.446" y2="5.08" width="0.3048" layer="1"/>
+<via x="12.446" y="5.08" extent="1-16" drill="0.5"/>
+<wire x1="12.446" y1="5.08" x2="12.446" y2="7.874" width="0.3048" layer="16"/>
+<via x="12.446" y="7.874" extent="1-16" drill="0.5"/>
+<wire x1="12.446" y1="7.874" x2="10.326" y2="9.74" width="0.3048" layer="1"/>
 <wire x1="10.326" y1="9.74" x2="8.89" y2="9.74" width="0.3048" layer="1"/>
 <wire x1="8.89" y1="9.74" x2="8.89" y2="10.16" width="0.3048" layer="1"/>
@@
 <wire x1="1.663" y1="1.27" x2="1.27" y2="1.663" width="0.3048" layer="1"/>
 </signal>
+<signal name="N$3">
+<contactref element="C9" pad="1"/>
+<contactref element="U$1" pad="20"/>
+<wire x1="65.698" y1="15.24" x2="67.83" y2="19.869" width="0" layer="19" extent="1-1"/>
+</signal>
+<signal name="N$4">
+<contactref element="C8" pad="1"/>
+<contactref element="U$1" pad="10"/>
+<wire x1="65.698" y1="11.938" x2="68.33" y2="23.819" width="0" layer="19" extent="1-1"/>
+</signal>
+<signal name="N$5">
+<contactref element="SJ1" pad="2"/>
+<contactref element="U$1" pad="9"/>
+<wire x1="60.452" y1="24.638" x2="68.83" y2="23.819" width="0" layer="19" extent="1-1"/>
+</signal>
 </signals>
