File: Flight-Controller-PCB1/flight-controller.brd (EAGLE design)
At the start: 79.9 x 27.9 mm, 45 parts, among them J1 1981584-1, U1 MK20DX256VLH7, U2 TPS61200, U3 MINI54TAN, Y1 32.768KHz, Y2 16Mhz/8pF

Commit message: finished teensy + imbue
Routing:
- net SCL: track 8.43 -> 44.6 mm, vias 2 -> 4
- net SDA: track 4.92 -> 30.9 mm, vias 0 -> 4
- net GND: track 223.2 -> 226.5 mm
- net RESET_B: track 28.0 -> 26.1 mm
Changed lines of the file:
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@@
 <wire x1="65.024" y1="21.082" x2="66.593" y2="21.082" width="0.254" layer="1"/>
 <wire x1="66.593" y1="21.082" x2="66.605" y2="21.094" width="0.254" layer="1"/>
-<wire x1="67.398" y1="15.24" x2="67.398" y2="11.938" width="0" layer="19" extent="1-1"/>
 <wire x1="66.605" y1="21.094" x2="66.605" y2="20.594" width="0.254" layer="1"/>
 <wire x1="66.605" y1="21.094" x2="65.036" y2="21.094" width="0.254" layer="1"/>
@@
 <wire x1="65.278" y1="22.098" x2="66.601" y2="22.098" width="0.254" layer="1"/>
 <wire x1="66.601" y1="22.098" x2="66.605" y2="22.094" width="0.254" layer="1"/>
+<wire x1="67.398" y1="11.938" x2="67.398" y2="15.24" width="0.254" layer="1"/>
 </signal>
 <signal name="N$2">
@@
 <wire x1="34.544" y1="-0.508" x2="52.832" y2="-0.508" width="0.254" layer="1"/>
 <wire x1="52.832" y1="-0.508" x2="54.102" y2="0.762" width="0.254" layer="1"/>
-<wire x1="54.102" y1="0.762" x2="54.102" y2="6.096" width="0.254" layer="1"/>
-<via x="54.102" y="6.096" extent="1-16" drill="0.5"/>
-<wire x1="54.102" y1="6.096" x2="54.102" y2="9.652" width="0.254" layer="16"/>
+<wire x1="54.102" y1="0.762" x2="54.102" y2="5.334" width="0.254" layer="1"/>
+<via x="54.102" y="5.334" extent="1-16" drill="0.5"/>
+<wire x1="54.102" y1="5.334" x2="54.102" y2="9.652" width="0.254" layer="16"/>
 <wire x1="54.102" y1="9.652" x2="50.038" y2="13.716" width="0.254" layer="16"/>
 <via x="50.038" y="13.716" extent="1-16" drill="0.5"/>
@@
 <wire x1="69.85" y1="18.542" x2="69.85" y2="19.849" width="0.254" layer="1"/>
 <wire x1="69.85" y1="19.849" x2="69.83" y2="19.869" width="0.254" layer="1"/>
-<wire x1="52.09" y1="8.27" x2="70.524" y2="15.24" width="0" layer="19" extent="1-1"/>
+<wire x1="70.524" y1="15.24" x2="69.596" y2="15.24" width="0.254" layer="1"/>
+<wire x1="69.596" y1="15.24" x2="67.818" y2="13.462" width="0.254" layer="1"/>
+<wire x1="67.818" y1="13.462" x2="66.294" y2="13.462" width="0.254" layer="1"/>
+<via x="66.294" y="13.462" extent="1-16" drill="0.5"/>
+<wire x1="66.294" y1="13.462" x2="64.77" y2="13.462" width="0.254" layer="16"/>
+<wire x1="64.77" y1="13.462" x2="64.008" y2="12.7" width="0.254" layer="16"/>
+<via x="64.008" y="12.7" extent="1-16" drill="0.5"/>
+<wire x1="64.008" y1="12.7" x2="62.23" y2="12.7" width="0.254" layer="1"/>
+<wire x1="62.23" y1="12.7" x2="61.722" y2="13.208" width="0.254" layer="1"/>
+<via x="61.722" y="13.208" extent="1-16" drill="0.5"/>
+<wire x1="61.722" y1="13.208" x2="61.722" y2="9.906" width="0.254" layer="16"/>
+<wire x1="61.722" y1="9.906" x2="59.182" y2="7.366" width="0.254" layer="16"/>
+<wire x1="59.182" y1="7.366" x2="55.88" y2="7.366" width="0.254" layer="16"/>
+<wire x1="55.88" y1="7.366" x2="54.864" y2="6.35" width="0.254" layer="16"/>
+<via x="54.864" y="6.35" extent="1-16" drill="0.5"/>
+<wire x1="54.864" y1="6.35" x2="52.832" y2="6.35" width="0.254" layer="1"/>
+<wire x1="52.832" y1="6.35" x2="52.07" y2="7.112" width="0.254" layer="1"/>
+<wire x1="52.07" y1="7.112" x2="52.07" y2="8.25" width="0.254" layer="1"/>
+<wire x1="52.07" y1="8.25" x2="52.09" y2="8.27" width="0.254" layer="1"/>
 </signal>
 <signal name="SCL">
@@
 <wire x1="69.342" y1="17.272" x2="69.342" y2="19.857" width="0.254" layer="1"/>
 <wire x1="69.342" y1="19.857" x2="69.33" y2="19.869" width="0.254" layer="1"/>
-<wire x1="51.59" y1="8.27" x2="69.342" y2="13.716" width="0" layer="19" extent="1-16"/>
+<wire x1="69.342" y1="13.716" x2="68.834" y2="13.208" width="0.254" layer="1"/>
+<wire x1="68.834" y1="13.208" x2="68.834" y2="2.286" width="0.254" layer="1"/>
+<wire x1="68.834" y1="2.286" x2="66.548" y2="0" width="0.254" layer="1"/>
+<wire x1="66.548" y1="0" x2="54.864" y2="0" width="0.254" layer="1"/>
+<via x="54.864" y="0" extent="1-16" drill="0.5"/>
+<wire x1="54.864" y1="0" x2="51.816" y2="3.048" width="0.254" layer="16"/>
+<wire x1="51.816" y1="3.048" x2="51.816" y2="6.096" width="0.254" layer="16"/>
+<via x="51.816" y="6.096" extent="1-16" drill="0.5"/>
+<wire x1="51.816" y1="6.096" x2="51.59" y2="6.322" width="0.254" layer="1"/>
+<wire x1="51.59" y1="6.322" x2="51.59" y2="8.27" width="0.254" layer="1"/>
 </signal>
 <signal name="N$19">
@@
 <wire x1="30.988" y1="8.89" x2="30.988" y2="7.112" width="0.254" layer="16"/>
 <wire x1="30.988" y1="7.112" x2="32.004" y2="6.096" width="0.254" layer="16"/>
-<wire x1="32.004" y1="6.096" x2="51.562" y2="6.096" width="0.254" layer="16"/>
-<via x="51.562" y="6.096" extent="1-16" drill="0.5"/>
-<wire x1="51.562" y1="6.096" x2="51.562" y2="6.604" width="0.254" layer="1"/>
-<wire x1="51.562" y1="6.604" x2="51.308" y2="6.858" width="0.254" layer="1"/>
-<wire x1="51.308" y1="6.858" x2="50.546" y2="6.858" width="0.254" layer="1"/>
-<wire x1="50.546" y1="6.858" x2="50.038" y2="7.366" width="0.254" layer="1"/>
-<wire x1="50.038" y1="7.366" x2="50.038" y2="8.218" width="0.254" layer="1"/>
+<wire x1="32.004" y1="6.096" x2="50.546" y2="6.096" width="0.254" layer="16"/>
+<via x="50.546" y="6.096" extent="1-16" drill="0.5"/>
+<wire x1="50.546" y1="6.096" x2="50.546" y2="6.35" width="0.254" layer="1"/>
+<wire x1="50.546" y1="6.35" x2="50.038" y2="6.858" width="0.254" layer="1"/>
+<wire x1="50.038" y1="6.858" x2="50.038" y2="8.218" width="0.254" layer="1"/>
 <wire x1="50.038" y1="8.218" x2="50.09" y2="8.27" width="0.254" layer="1"/>
 </signal>

Commit message: working on arduino pro mini
Parts:
- added C12, C13: 0.1uF, SparkFun:0603-CAP
- added D3: Green, Testing:0603-LED-ALT1
- added JP1: FTDI Basic, SparkFun:1X06
- added Q1: 8/16/20MHz, Testing:RESONATOR-SMD-1:1
- added R11: 330, SparkFun:0603-RES
- added R12, R13: (no value), SparkFun:0603-RES
- added R8: 10K, SparkFun:0603-RES
- added S1: Reset, Testing:TACTILE-SWITCH-SMD-ALT01
- added U4: ATMEGA328, SparkFun:TQFP32-08
Connections:
- new net A4: R12.1, U4.27
- new net A5: R13.1, U4.28
- new net AREF: C12.2, U4.20
- new net DTR: C13.2, JP1.1
- new net N$6: Q1.3, U4.8
- new net N$7: D3.A, R11.2
- new net N$8: Q1.1, U4.7
- new net RESET: C13.1, R8.1, S1.3, S1.4, U4.29
- new net RXI: JP1.3
- new net TXO: JP1.2
- net 3.3V: now also R12.2, R13.2, R8.2, U4.18, U4.4, U4.6
- net GND: now also C12.1, D3.C, JP1.5, JP1.6, Q1.2, S1.1, S1.2, U4.21, U4.3, U4.5
- net SCK: now also R11.1, U4.17
- net VCC: now also JP1.4
Changed lines of the file:
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@@
 <?xml version="1.0" encoding="utf-8"?>
 <!DOCTYPE eagle SYSTEM "eagle.dtd">
-<eagle version="7.4.0">
+<eagle version="7.5.0">
 <drawing>
 <settings>
@@
 <attribute name="MF" value="Panasonic" x="71.374" y="11.938" size="1.778" layer="27" rot="R180" display="off"/>
 </element>
+<element name="R8" library="SparkFun" package="0603-RES" value="10K" x="13.97" y="-20.32"/>
+<element name="C12" library="SparkFun" package="0603-CAP" value="0.1uF" x="7.874" y="-20.32"/>
+<element name="R11" library="SparkFun" package="0603-RES" value="330" x="-2.794" y="-24.384"/>
+<element name="D3" library="Testing" package="0603-LED-ALT1" value="Green" x="1.524" y="-20.574"/>
+<element name="U4" library="SparkFun" package="TQFP32-08" value="ATMEGA328" x="0.762" y="-7.112"/>
+<element name="C13" library="SparkFun" package="0603-CAP" value="0.1uF" x="10.922" y="-20.32"/>
+<element name="R12" library="SparkFun" package="0603-RES" value="" x="0.254" y="-24.384"/>
+<element name="R13" library="SparkFun" package="0603-RES" value="" x="3.302" y="-24.384"/>
+<element name="S1" library="Testing" package="TACTILE-SWITCH-SMD-ALT01" value="Reset" x="9.652" y="-4.064"/>
+<element name="Q1" library="Testing" package="RESONATOR-SMD-1:1" value="8/16/20MHz" x="-2.286" y="-20.828"/>
+<element name="JP1" library="SparkFun" package="1X06" value="FTDI Basic" x="-2.54" y="-29.718"/>
 </elements>
 <signals>
@@
 <wire x1="66.601" y1="22.098" x2="66.605" y2="22.094" width="0.254" layer="1"/>
 <wire x1="67.398" y1="11.938" x2="67.398" y2="15.24" width="0.254" layer="1"/>
+<contactref element="S1" pad="1"/>
+<contactref element="S1" pad="2"/>
+<contactref element="C12" pad="1"/>
+<contactref element="D3" pad="C"/>
+<contactref element="Q1" pad="2"/>
+<contactref element="U4" pad="5"/>
+<contactref element="U4" pad="3"/>
+<contactref element="U4" pad="21"/>
+<contactref element="JP1" pad="5"/>
+<contactref element="JP1" pad="6"/>
+<wire x1="10.16" y1="-29.718" x2="7.62" y2="-29.718" width="0" layer="19" extent="1-1"/>
+<wire x1="7.024" y1="-20.32" x2="7.62" y2="-29.718" width="0" layer="19" extent="1-1"/>
+<wire x1="1.524" y1="-19.697" x2="7.024" y2="-20.32" width="0" layer="19" extent="1-1"/>
+<wire x1="-2.286" y1="-19.812" x2="1.524" y2="-19.697" width="0" layer="19" extent="1-1"/>
+<wire x1="-3.5306" y1="-7.512" x2="-2.286" y2="-19.812" width="0" layer="19" extent="1-1"/>
+<wire x1="-3.5306" y1="-5.912" x2="-3.5306" y2="-7.512" width="0" layer="19" extent="1-1"/>
+<wire x1="5.0546" y1="-6.712" x2="-3.5306" y2="-7.512" width="0" layer="19" extent="1-1"/>
+<wire x1="6.858" y1="-2.159" x2="5.0546" y2="-6.712" width="0" layer="19" extent="1-1"/>
+<wire x1="6.858" y1="-0.254" x2="6.858" y2="-2.159" width="0" layer="19" extent="1-1"/>
+<wire x1="12.446" y1="-2.159" x2="13.208" y2="-0.254" width="0" layer="19" extent="1-1"/>
 </signal>
 <signal name="N$2">
@@
 <wire x1="54.864" y1="17.526" x2="54.864" y2="16.764" width="0.254" layer="1"/>
 <wire x1="54.864" y1="16.764" x2="55.88" y2="15.748" width="0.254" layer="1"/>
+<contactref element="U4" pad="18"/>
+<contactref element="U4" pad="4"/>
+<contactref element="U4" pad="6"/>
+<contactref element="R12" pad="2"/>
+<contactref element="R13" pad="2"/>
+<contactref element="R8" pad="2"/>
+<wire x1="4.152" y1="-24.384" x2="1.104" y2="-24.384" width="0" layer="19" extent="1-1"/>
+<wire x1="14.82" y1="-20.32" x2="4.152" y2="-24.384" width="0" layer="19" extent="1-1"/>
+<wire x1="5.0546" y1="-9.112" x2="14.82" y2="-20.32" width="0" layer="19" extent="1-1"/>
+<wire x1="-3.5306" y1="-8.312" x2="5.0546" y2="-9.112" width="0" layer="19" extent="1-1"/>
+<wire x1="-3.5306" y1="-6.712" x2="-3.5306" y2="-8.312" width="0" layer="19" extent="1-1"/>
+<wire x1="1.27" y1="3.417" x2="-3.5306" y2="-6.712" width="0" layer="19" extent="1-1"/>
 </signal>
 <signal name="PS">
@@
 <signal name="SCK">
 <contactref element="U1" pad="50"/>
+<contactref element="U4" pad="17"/>
+<contactref element="R11" pad="1"/>
+<wire x1="5.0546" y1="-9.912" x2="59.04" y2="10.72" width="0" layer="19" extent="1-1"/>
+<wire x1="-3.644" y1="-24.384" x2="5.0546" y2="-9.912" width="0" layer="19" extent="1-1"/>
 </signal>
 <signal name="SWD_DIO">
@@
 <wire x1="19.47" y1="22.86" x2="20.32" y2="22.01" width="0.254" layer="1"/>
 <wire x1="20.32" y1="22.01" x2="22.86" y2="22.01" width="0.4064" layer="1"/>
+<contactref element="JP1" pad="4"/>
+<wire x1="6.35" y1="-0.254" x2="5.08" y2="-29.718" width="0" layer="19" extent="16-16"/>
 </signal>
 <signal name="N$12">
@@
 <wire x1="68.834" y1="23.823" x2="68.83" y2="23.819" width="0.254" layer="1"/>
 </signal>
+<signal name="AREF">
+<contactref element="C12" pad="2"/>
+<contactref element="U4" pad="20"/>
+<wire x1="5.0546" y1="-7.512" x2="8.724" y2="-20.32" width="0" layer="19" extent="1-1"/>
+</signal>
+<signal name="RESET">
+<contactref element="U4" pad="29"/>
+<contactref element="R8" pad="1"/>
+<contactref element="C13" pad="1"/>
+<contactref element="S1" pad="3"/>
+<contactref element="S1" pad="4"/>
+<wire x1="13.12" y1="-20.32" x2="10.072" y2="-20.32" width="0" layer="19" extent="1-1"/>
+<wire x1="12.446" y1="-5.969" x2="13.12" y2="-20.32" width="0" layer="19" extent="1-1"/>
+<wire x1="6.858" y1="-5.969" x2="12.446" y2="-5.969" width="0" layer="19" extent="1-1"/>
+<wire x1="0.362" y1="-2.8194" x2="6.858" y2="-5.969" width="0" layer="19" extent="1-1"/>
+</signal>
+<signal name="N$7">
+<contactref element="R11" pad="2"/>
+<contactref element="D3" pad="A"/>
+<wire x1="1.524" y1="-21.451" x2="-1.944" y2="-24.384" width="0" layer="19" extent="1-1"/>
+</signal>
+<signal name="A5">
+<contactref element="U4" pad="28"/>
+<contactref element="R13" pad="1"/>
+<wire x1="1.162" y1="-2.8194" x2="2.452" y2="-24.384" width="0" layer="19" extent="1-1"/>
+</signal>
+<signal name="A4">
+<contactref element="U4" pad="27"/>
+<contactref element="R12" pad="1"/>
+<wire x1="1.962" y1="-2.8194" x2="-0.596" y2="-24.384" width="0" layer="19" extent="1-1"/>
+</signal>
+<signal name="N$6">
+<contactref element="U4" pad="8"/>
+<contactref element="Q1" pad="3"/>
+<wire x1="-3.5306" y1="-9.912" x2="-1.086" y2="-19.812" width="0" layer="19" extent="1-1"/>
+</signal>
+<signal name="N$8">
+<contactref element="U4" pad="7"/>
+<contactref element="Q1" pad="1"/>
+<wire x1="-3.5306" y1="-9.112" x2="-3.486" y2="-19.812" width="0" layer="19" extent="1-1"/>
+</signal>
+<signal name="DTR">
+<contactref element="C13" pad="2"/>
+<contactref element="JP1" pad="1"/>
+<wire x1="11.772" y1="-20.32" x2="-2.54" y2="-29.718" width="0" layer="19" extent="1-1"/>
+</signal>
+<signal name="TXO">
+<contactref element="JP1" pad="2"/>
+</signal>
+<signal name="RXI">
+<contactref element="JP1" pad="3"/>
+</signal>
 </signals>

Commit message: still working on microcontroller
Connections:
- removed net RXI: JP1.3
- removed net TXO: JP1.2
- new net N$10: JP1.2, U4.31
- new net N$9: JP1.3, U4.30
- net 3.3V: now also JP1.4
- net VCC: no longer JP1.4
Changed lines of the file:
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@@
 <contactref element="R13" pad="2"/>
 <contactref element="R8" pad="2"/>
+<contactref element="JP1" pad="4"/>
 <wire x1="4.152" y1="-24.384" x2="1.104" y2="-24.384" width="0" layer="19" extent="1-1"/>
+<wire x1="5.08" y1="-29.718" x2="4.152" y2="-24.384" width="0" layer="19" extent="1-1"/>
 <wire x1="14.82" y1="-20.32" x2="4.152" y2="-24.384" width="0" layer="19" extent="1-1"/>
 <wire x1="5.0546" y1="-9.112" x2="14.82" y2="-20.32" width="0" layer="19" extent="1-1"/>
@@
 <wire x1="19.47" y1="22.86" x2="20.32" y2="22.01" width="0.254" layer="1"/>
 <wire x1="20.32" y1="22.01" x2="22.86" y2="22.01" width="0.4064" layer="1"/>
-<contactref element="JP1" pad="4"/>
-<wire x1="6.35" y1="-0.254" x2="5.08" y2="-29.718" width="0" layer="19" extent="16-16"/>
 </signal>
 <signal name="N$12">
@@
 <wire x1="11.772" y1="-20.32" x2="-2.54" y2="-29.718" width="0" layer="19" extent="1-1"/>
 </signal>
-<signal name="TXO">
+<signal name="N$9">
+<contactref element="JP1" pad="3"/>
+<contactref element="U4" pad="30"/>
+<wire x1="-0.438" y1="-2.8194" x2="2.54" y2="-29.718" width="0" layer="19" extent="1-1"/>
+</signal>
+<signal name="N$10">
 <contactref element="JP1" pad="2"/>
-</signal>
-<signal name="RXI">
-<contactref element="JP1" pad="3"/>
+<contactref element="U4" pad="31"/>
+<wire x1="-1.238" y1="-2.8194" x2="0" y2="-29.718" width="0" layer="19" extent="1-1"/>
 </signal>
 </signals>

Commit message: laying out board for final time
Parts:
- removed R12, R13: (no value), SparkFun:0603-RES
- moved JP1 92.8 mm to (75.9, 19.8), turned to 90 degrees
- moved R11 82.2 mm to (58.4, 30.5)
- moved D3 79.6 mm to (58.4, 35.1)
- moved C12 76.0 mm to (55.9, 38.6), turned to 180 degrees
- moved R8 73.1 mm to (62.0, 34.8), turned to 90 degrees
- moved C13 72.6 mm to (62.7, 30.5)
- moved Q1 68.6 mm to (42.9, 30.7), turned to 270 degrees
- moved S1 65.5 mm to (74.7, 3.81)
- moved U4 64.1 mm to (51.3, 32.3)
Connections:
- removed net A4: R12.1, U4.27
- removed net A5: R13.1, U4.28
- new net NONE: R11.1, U4.17
- net 3.3V: no longer R12.2, R13.2
- net SCK: no longer R11.1, U4.17
- net SCL: now also U4.28
- net SDA: now also U4.27
Other:
- board size 79.9 x 27.9 mm -> 79.9 x 42.9 mm
- board text added: "Based off: Teensy 3.1 by Paul Stoffregen and Arduino Pro Mini by Team Arduino"
- board text added: "Designed by: Kevin Sheridan and Casimir Duchnowski"
- board text added: "GND"
- board text added: "Purdue AUVSI IARC Team Flight Controller 2016"
