File: Flight-Controller-PCB1/flight-controller.brd (EAGLE design)
At the start: 79.9 x 42.9 mm, 54 parts, among them J1 1981584-1, Q1 8/16/20MHz, U1 MK20DX256VLH7, U2 TPS61200, U3 MINI54TAN, U4 ATMEGA328, Y1 32.768KHz, Y2 16Mhz/8pF

Commit message: making mods to pins
Parts:
- added JP2, JP3, JP4, JP5, JP6, JP7: (no value), adafruit:1X03
- moved R8 5.29 mm to (58.9, 39.1)
- moved D3 4.93 mm to (55.6, 39.1)
- moved R11 4.68 mm to (59.4, 35.1)
- moved C12 4.44 mm to (51.6, 39.6)
- moved C13 3.75 mm to (59.4, 28.7)
- moved JP1 3.05 mm to (75.9, 16.8)
Connections:
- net GND: now also JP2.1, JP3.1, JP4.1, JP5.1, JP6.1, JP7.1
- net SCL: now also JP2.2, JP3.2, JP4.2, JP5.2, JP6.2, JP7.2
- net SDA: now also JP2.3, JP3.3, JP4.3, JP5.3, JP6.3, JP7.3
Other:
- board text added: "I2C"
- board text added: "SDA SCL GND"

Commit message: wiring attempting
Parts:
- added JP10, JP11, JP8, JP9: (no value), adafruit:1X03
- moved D3 3.88 mm to (53.6, 35.8)
- moved U4 3.75 mm to (48.0, 30.5)
- moved Q1 3.61 mm to (40.6, 27.9)
- moved R11 2.55 mm to (56.9, 35.3)
- moved R8 2.54 mm to (56.4, 39.1)
- moved C13 2.50 mm to (57.1, 29.7)
- moved C12 0.25 mm to (51.6, 39.9)
Connections:
- new net N$11: JP10.3, U4.32
- new net N$13: JP9.3, U4.1
- new net N$14: JP8.3, U4.2
- new net N$16: JP11.3, U4.9
- net GND: now also JP10.1, JP11.1, JP8.1, JP9.1
Routing:
- net GND: track 226.5 -> 373.2 mm, vias 15 -> 19
- net SCL: track 44.8 -> 107.5 mm, vias 4 -> 6
- net 3.3V: track 206.5 -> 260.9 mm, vias 11 -> 14
- net SDA: track 30.9 -> 80.0 mm, vias 4 -> 5
- net N$16: track 0.00 -> 35.3 mm
- net NONE: track 0.00 -> 12.0 mm, vias 0 -> 2
- net N$7: track 0.00 -> 7.35 mm, vias 0 -> 2
- net N$6: track 0.00 -> 2.45 mm
- net N$8: track 0.00 -> 2.36 mm
Other:
- board text added: "GND VCC SIG"
- board text added: "PWM IN"

Commit message: Ready for manufacturer
Routing:
- net N$10: track 0.00 -> 105.8 mm, vias 0 -> 9
- net N$9: track 0.00 -> 93.1 mm, vias 0 -> 5
- net RESET: track 0.00 -> 80.6 mm, vias 0 -> 4
- net SCL: track 107.5 -> 155.1 mm
- net DTR: track 0.00 -> 43.8 mm
- net SDA: track 80.0 -> 121.4 mm, vias 5 -> 7
- net GND: track 373.2 -> 404.2 mm, vias 19 -> 21
- net N$13: track 0.00 -> 27.4 mm, vias 0 -> 1
- net N$14: track 0.00 -> 27.4 mm, vias 0 -> 1
- net N$11: track 0.00 -> 24.8 mm, vias 0 -> 1
- net AREF: track 0.00 -> 12.7 mm, vias 0 -> 2
- net N$19: track 22.5 -> 23.2 mm
- net VREFH: track 35.6 -> 34.9 mm
- net N$2: track 10.8 -> 10.2 mm
