File: Hardware/Flight-Controller-PCB1/flight-controller.sch (EAGLE design)
At the start: 55 parts, among them J1 1981584-1, Q1 8/16/20MHz, U1 MK20DX256VLH7, U2 TPS61200, U3 MINI54TAN, U4 ATMEGA328, Y1 32.768KHz, Y2 16Mhz/8pF

Commit message: firmware
Parts:
- added JP10, JP11, JP3, JP4, JP5, JP6, JP7, JP8, JP9: (no value), adafruit:PINHD-1X3
Connections:
- new net N$11: JP10.3, U4.PD2(INT0)
- new net N$13: JP9.3, U4.PD3(INT1)
- new net N$14: JP8.3, U4.PD4(XCK/T0)
- new net N$16: JP11.3, U4.PD5(T1)
- net GND: now also JP10.1, JP11.1, JP3.1, JP4.1, JP5.1, JP6.1, JP7.1, JP8.1, JP9.1
- net SCL: now also JP2.2, JP3.2, JP4.2, JP5.2, JP6.2, JP7.2
- net SDA: now also JP3.3, JP4.3, JP5.3, JP6.3, JP7.3
Changed lines of the file:
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@@
 <part name="JP2" library="adafruit" deviceset="PINHD-1X3" device=""/>
 <part name="GND15" library="supply1" deviceset="GND" device=""/>
+<part name="JP3" library="adafruit" deviceset="PINHD-1X3" device=""/>
+<part name="GND20" library="supply1" deviceset="GND" device=""/>
+<part name="JP4" library="adafruit" deviceset="PINHD-1X3" device=""/>
+<part name="GND21" library="supply1" deviceset="GND" device=""/>
+<part name="JP5" library="adafruit" deviceset="PINHD-1X3" device=""/>
+<part name="GND22" library="supply1" deviceset="GND" device=""/>
+<part name="JP6" library="adafruit" deviceset="PINHD-1X3" device=""/>
+<part name="GND23" library="supply1" deviceset="GND" device=""/>
+<part name="JP7" library="adafruit" deviceset="PINHD-1X3" device=""/>
+<part name="GND24" library="supply1" deviceset="GND" device=""/>
+<part name="JP8" library="adafruit" deviceset="PINHD-1X3" device=""/>
+<part name="GND25" library="supply1" deviceset="GND" device=""/>
+<part name="JP9" library="adafruit" deviceset="PINHD-1X3" device=""/>
+<part name="GND26" library="supply1" deviceset="GND" device=""/>
+<part name="JP10" library="adafruit" deviceset="PINHD-1X3" device=""/>
+<part name="GND27" library="supply1" deviceset="GND" device=""/>
+<part name="JP11" library="adafruit" deviceset="PINHD-1X3" device=""/>
+<part name="GND28" library="supply1" deviceset="GND" device=""/>
 </parts>
 <sheets>
@@
 <instance part="JP2" gate="A" x="-40.64" y="20.32" rot="R180"/>
 <instance part="GND15" gate="1" x="-30.48" y="17.78" rot="R90"/>
+<instance part="JP3" gate="A" x="-40.64" y="2.54" rot="R180"/>
+<instance part="GND20" gate="1" x="-30.48" y="0" rot="R90"/>
+<instance part="JP4" gate="A" x="-5.08" y="20.32" rot="R180"/>
+<instance part="GND21" gate="1" x="5.08" y="17.78" rot="R90"/>
+<instance part="JP5" gate="A" x="-5.08" y="2.54" rot="R180"/>
+<instance part="GND22" gate="1" x="5.08" y="0" rot="R90"/>
+<instance part="JP6" gate="A" x="-22.86" y="-15.24" rot="R180"/>
+<instance part="GND23" gate="1" x="-12.7" y="-17.78" rot="R90"/>
+<instance part="JP7" gate="A" x="-22.86" y="-33.02" rot="R180"/>
+<instance part="GND24" gate="1" x="-12.7" y="-35.56" rot="R90"/>
+<instance part="JP8" gate="A" x="27.94" y="-20.32"/>
+<instance part="GND25" gate="1" x="17.78" y="-17.78" rot="R270"/>
+<instance part="JP9" gate="A" x="27.94" y="-35.56"/>
+<instance part="GND26" gate="1" x="17.78" y="-33.02" rot="R270"/>
+<instance part="JP10" gate="A" x="27.94" y="-50.8"/>
+<instance part="GND27" gate="1" x="17.78" y="-48.26" rot="R270"/>
+<instance part="JP11" gate="A" x="27.94" y="-2.54"/>
+<instance part="GND28" gate="1" x="17.78" y="0" rot="R270"/>
 </instances>
 <busses>
@@
 <pinref part="JP2" gate="A" pin="1"/>
 <wire x1="-33.02" y1="17.78" x2="-38.1" y2="17.78" width="0.1524" layer="91"/>
+</segment>
+<segment>
+<pinref part="GND20" gate="1" pin="GND"/>
+<pinref part="JP3" gate="A" pin="1"/>
+<wire x1="-33.02" y1="0" x2="-38.1" y2="0" width="0.1524" layer="91"/>
+</segment>
+<segment>
+<pinref part="GND21" gate="1" pin="GND"/>
+<pinref part="JP4" gate="A" pin="1"/>
+<wire x1="2.54" y1="17.78" x2="-2.54" y2="17.78" width="0.1524" layer="91"/>
+</segment>
+<segment>
+<pinref part="GND22" gate="1" pin="GND"/>
+<pinref part="JP5" gate="A" pin="1"/>
+<wire x1="2.54" y1="0" x2="-2.54" y2="0" width="0.1524" layer="91"/>
+</segment>
+<segment>
+<pinref part="GND23" gate="1" pin="GND"/>
+<pinref part="JP6" gate="A" pin="1"/>
+<wire x1="-15.24" y1="-17.78" x2="-20.32" y2="-17.78" width="0.1524" layer="91"/>
+</segment>
+<segment>
+<pinref part="GND24" gate="1" pin="GND"/>
+<pinref part="JP7" gate="A" pin="1"/>
+<wire x1="-15.24" y1="-35.56" x2="-20.32" y2="-35.56" width="0.1524" layer="91"/>
+</segment>
+<segment>
+<pinref part="JP8" gate="A" pin="1"/>
+<pinref part="GND25" gate="1" pin="GND"/>
+<wire x1="25.4" y1="-17.78" x2="20.32" y2="-17.78" width="0.1524" layer="91"/>
+</segment>
+<segment>
+<pinref part="JP9" gate="A" pin="1"/>
+<pinref part="GND26" gate="1" pin="GND"/>
+<wire x1="25.4" y1="-33.02" x2="20.32" y2="-33.02" width="0.1524" layer="91"/>
+</segment>
+<segment>
+<pinref part="JP10" gate="A" pin="1"/>
+<pinref part="GND27" gate="1" pin="GND"/>
+<wire x1="25.4" y1="-48.26" x2="20.32" y2="-48.26" width="0.1524" layer="91"/>
+</segment>
+<segment>
+<pinref part="JP11" gate="A" pin="1"/>
+<pinref part="GND28" gate="1" pin="GND"/>
+<wire x1="25.4" y1="0" x2="20.32" y2="0" width="0.1524" layer="91"/>
 </segment>
 </net>
@@
 <label x="-30.48" y="22.86" size="1.778" layer="95"/>
 </segment>
+<segment>
+<pinref part="JP3" gate="A" pin="3"/>
+<wire x1="-38.1" y1="5.08" x2="-30.48" y2="5.08" width="0.1524" layer="91"/>
+<label x="-30.48" y="5.08" size="1.778" layer="95"/>
+</segment>
+<segment>
+<pinref part="JP4" gate="A" pin="3"/>
+<wire x1="-2.54" y1="22.86" x2="5.08" y2="22.86" width="0.1524" layer="91"/>
+<label x="5.08" y="22.86" size="1.778" layer="95"/>
+</segment>
+<segment>
+<pinref part="JP5" gate="A" pin="3"/>
+<wire x1="-2.54" y1="5.08" x2="5.08" y2="5.08" width="0.1524" layer="91"/>
+<label x="5.08" y="5.08" size="1.778" layer="95"/>
+</segment>
+<segment>
+<pinref part="JP6" gate="A" pin="3"/>
+<wire x1="-20.32" y1="-12.7" x2="-12.7" y2="-12.7" width="0.1524" layer="91"/>
+<label x="-12.7" y="-12.7" size="1.778" layer="95"/>
+</segment>
+<segment>
+<pinref part="JP7" gate="A" pin="3"/>
+<wire x1="-20.32" y1="-30.48" x2="-12.7" y2="-30.48" width="0.1524" layer="91"/>
+<label x="-12.7" y="-30.48" size="1.778" layer="95"/>
+</segment>
 </net>
 <net name="SCL" class="0">
@@
 <segment>
 <pinref part="U4" gate="G$1" pin="PC5(ADC5/SCL)"/>
-<wire x1="7.62" y1="-66.04" x2="27.94" y2="-66.04" width="0.1524" layer="91"/>
-</segment>
-<segment>
-<wire x1="-40.64" y1="20.32" x2="-45.72" y2="20.32" width="0.1524" layer="91"/>
+<wire x1="7.62" y1="-66.04" x2="25.4" y2="-66.04" width="0.1524" layer="91"/>
+<label x="25.4" y="-66.04" size="1.778" layer="95"/>
+</segment>
+<segment>
+<wire x1="-38.1" y1="20.32" x2="-45.72" y2="20.32" width="0.1524" layer="91"/>
 <label x="-50.8" y="20.32" size="1.778" layer="95"/>
+<pinref part="JP2" gate="A" pin="2"/>
+</segment>
+<segment>
+<wire x1="-38.1" y1="2.54" x2="-45.72" y2="2.54" width="0.1524" layer="91"/>
+<label x="-50.8" y="2.54" size="1.778" layer="95"/>
+<pinref part="JP3" gate="A" pin="2"/>
+</segment>
+<segment>
+<wire x1="-2.54" y1="20.32" x2="-10.16" y2="20.32" width="0.1524" layer="91"/>
+<label x="-15.24" y="20.32" size="1.778" layer="95"/>
+<pinref part="JP4" gate="A" pin="2"/>
+</segment>
+<segment>
+<wire x1="-2.54" y1="2.54" x2="-10.16" y2="2.54" width="0.1524" layer="91"/>
+<label x="-15.24" y="2.54" size="1.778" layer="95"/>
+<pinref part="JP5" gate="A" pin="2"/>
+</segment>
+<segment>
+<wire x1="-20.32" y1="-15.24" x2="-27.94" y2="-15.24" width="0.1524" layer="91"/>
+<label x="-33.02" y="-15.24" size="1.778" layer="95"/>
+<pinref part="JP6" gate="A" pin="2"/>
+</segment>
+<segment>
+<wire x1="-20.32" y1="-33.02" x2="-27.94" y2="-33.02" width="0.1524" layer="91"/>
+<label x="-33.02" y="-33.02" size="1.778" layer="95"/>
+<pinref part="JP7" gate="A" pin="2"/>
 </segment>
 </net>
@@
 </segment>
 </net>
+<net name="N$11" class="0">
+<segment>
+<pinref part="JP10" gate="A" pin="3"/>
+<wire x1="25.4" y1="-53.34" x2="30.48" y2="-53.34" width="0.1524" layer="91"/>
+<wire x1="30.48" y1="-53.34" x2="30.48" y2="-81.28" width="0.1524" layer="91"/>
+<pinref part="U4" gate="G$1" pin="PD2(INT0)"/>
+<wire x1="30.48" y1="-81.28" x2="7.62" y2="-81.28" width="0.1524" layer="91"/>
+</segment>
+</net>
+<net name="N$13" class="0">
+<segment>
+<pinref part="JP9" gate="A" pin="3"/>
+<wire x1="25.4" y1="-38.1" x2="33.02" y2="-38.1" width="0.1524" layer="91"/>
+<wire x1="33.02" y1="-38.1" x2="33.02" y2="-83.82" width="0.1524" layer="91"/>
+<pinref part="U4" gate="G$1" pin="PD3(INT1)"/>
+<wire x1="33.02" y1="-83.82" x2="7.62" y2="-83.82" width="0.1524" layer="91"/>
+</segment>
+</net>
+<net name="N$14" class="0">
+<segment>
+<pinref part="JP8" gate="A" pin="3"/>
+<wire x1="25.4" y1="-22.86" x2="35.56" y2="-22.86" width="0.1524" layer="91"/>
+<wire x1="35.56" y1="-22.86" x2="35.56" y2="-86.36" width="0.1524" layer="91"/>
+<pinref part="U4" gate="G$1" pin="PD4(XCK/T0)"/>
+<wire x1="35.56" y1="-86.36" x2="7.62" y2="-86.36" width="0.1524" layer="91"/>
+</segment>
+</net>
+<net name="N$16" class="0">
+<segment>
+<pinref part="JP11" gate="A" pin="3"/>
+<wire x1="25.4" y1="-5.08" x2="38.1" y2="-5.08" width="0.1524" layer="91"/>
+<wire x1="38.1" y1="-5.08" x2="38.1" y2="-88.9" width="0.1524" layer="91"/>
+<pinref part="U4" gate="G$1" pin="PD5(T1)"/>
+<wire x1="38.1" y1="-88.9" x2="7.62" y2="-88.9" width="0.1524" layer="91"/>
+</segment>
+</net>
