File: Hardware/Teensy-FC-BOB/Teensy-FC-BOB.sch (EAGLE design)
At the start: 21 parts, among them U1 MPU-9250, U3 BMP180;314030004

Commit message: finishing pins
Parts:
- added I2C1, I2C2, I2C3, I2C4, I2C5: GND-SDA-SCL, pinhead:PINHD-1X3
- added PWM6: PWMOUT4, pinhead:PINHD-1X3
- added PWM7: PWMOUT3, pinhead:PINHD-1X3
- added PWM8: PWMOUT2, pinhead:PINHD-1X3
- added PWM9: PWMOUT1, pinhead:PINHD-1X3
Connections:
- new net N$10: FLIGHTCONTROL.20/A6/PWM, PWM9.3
- new net N$11: FLIGHTCONTROL.21/A7/PWM, PWM8.3
- new net N$12: FLIGHTCONTROL.22/A8/T/PWM, PWM7.3
- new net N$13: FLIGHTCONTROL.23/A9/T/PWM, PWM6.3
- net GND: now also PWM6.1, PWM7.1, PWM8.1, PWM9.1
- net VCC_5V: now also PWM6.2, PWM7.2, PWM8.2, PWM9.2
Changed lines of the file:
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@@
 <part name="5V" library="pinhead" deviceset="PINHD-1X2" device="" value="5V"/>
 <part name="U$2" library="Power or GND " deviceset="GND_POWER" device=""/>
+<part name="PWM6" library="pinhead" deviceset="PINHD-1X3" device="" value="PWMOUT4"/>
+<part name="PWM7" library="pinhead" deviceset="PINHD-1X3" device="" value="PWMOUT3"/>
+<part name="PWM8" library="pinhead" deviceset="PINHD-1X3" device="" value="PWMOUT2"/>
+<part name="PWM9" library="pinhead" deviceset="PINHD-1X3" device="" value="PWMOUT1"/>
+<part name="U$3" library="Power or GND " deviceset="GND_POWER" device=""/>
+<part name="I2C1" library="pinhead" deviceset="PINHD-1X3" device="" value="GND-SDA-SCL"/>
+<part name="I2C2" library="pinhead" deviceset="PINHD-1X3" device="" value="GND-SDA-SCL"/>
+<part name="I2C3" library="pinhead" deviceset="PINHD-1X3" device="" value="GND-SDA-SCL"/>
+<part name="I2C4" library="pinhead" deviceset="PINHD-1X3" device="" value="GND-SDA-SCL"/>
+<part name="I2C5" library="pinhead" deviceset="PINHD-1X3" device="" value="GND-SDA-SCL"/>
 </parts>
 <sheets>
@@
 <instance part="5V" gate="G$1" x="76.2" y="154.94"/>
 <instance part="U$2" gate="G$1" x="55.88" y="165.1" rot="R180"/>
+<instance part="PWM6" gate="A" x="-132.08" y="0" rot="R180"/>
+<instance part="PWM7" gate="A" x="-132.08" y="17.78" rot="R180"/>
+<instance part="PWM8" gate="A" x="-132.08" y="35.56" rot="R180"/>
+<instance part="PWM9" gate="A" x="-132.08" y="53.34" rot="R180"/>
+<instance part="U$3" gate="G$1" x="-154.94" y="71.12" rot="R180"/>
+<instance part="I2C1" gate="A" x="101.6" y="157.48" rot="R90"/>
+<instance part="I2C2" gate="A" x="119.38" y="157.48" rot="R90"/>
+<instance part="I2C3" gate="A" x="137.16" y="157.48" rot="R90"/>
+<instance part="I2C4" gate="A" x="154.94" y="157.48" rot="R90"/>
+<instance part="I2C5" gate="A" x="172.72" y="157.48" rot="R90"/>
 </instances>
 <busses>
@@
 <label x="55.88" y="162.56" size="1.778" layer="95"/>
 </segment>
+<segment>
+<pinref part="PWM9" gate="A" pin="1"/>
+<pinref part="U$3" gate="G$1" pin="GND"/>
+<wire x1="-129.54" y1="50.8" x2="-154.94" y2="50.8" width="0.1524" layer="91"/>
+<wire x1="-154.94" y1="50.8" x2="-154.94" y2="71.12" width="0.1524" layer="91"/>
+<pinref part="PWM8" gate="A" pin="1"/>
+<wire x1="-129.54" y1="33.02" x2="-154.94" y2="33.02" width="0.1524" layer="91"/>
+<wire x1="-154.94" y1="33.02" x2="-154.94" y2="50.8" width="0.1524" layer="91"/>
+<pinref part="PWM7" gate="A" pin="1"/>
+<wire x1="-129.54" y1="15.24" x2="-154.94" y2="15.24" width="0.1524" layer="91"/>
+<wire x1="-154.94" y1="15.24" x2="-154.94" y2="33.02" width="0.1524" layer="91"/>
+<pinref part="PWM6" gate="A" pin="1"/>
+<wire x1="-129.54" y1="-2.54" x2="-154.94" y2="-2.54" width="0.1524" layer="91"/>
+<wire x1="-154.94" y1="-2.54" x2="-154.94" y2="15.24" width="0.1524" layer="91"/>
+<label x="-154.94" y="25.4" size="1.778" layer="95"/>
+</segment>
 </net>
 <net name="VCC_3V3" class="0">
@@
 <label x="55.88" y="154.94" size="1.778" layer="95"/>
 </segment>
+<segment>
+<pinref part="PWM9" gate="A" pin="2"/>
+<wire x1="-129.54" y1="53.34" x2="-116.84" y2="53.34" width="0.1524" layer="91"/>
+<label x="-116.84" y="53.34" size="1.778" layer="95"/>
+</segment>
+<segment>
+<pinref part="PWM8" gate="A" pin="2"/>
+<wire x1="-129.54" y1="35.56" x2="-116.84" y2="35.56" width="0.1524" layer="91"/>
+<label x="-116.84" y="35.56" size="1.778" layer="95"/>
+</segment>
+<segment>
+<pinref part="PWM7" gate="A" pin="2"/>
+<wire x1="-129.54" y1="17.78" x2="-116.84" y2="17.78" width="0.1524" layer="91"/>
+<label x="-116.84" y="17.78" size="1.778" layer="95"/>
+</segment>
+<segment>
+<pinref part="PWM6" gate="A" pin="2"/>
+<wire x1="-129.54" y1="0" x2="-116.84" y2="0" width="0.1524" layer="91"/>
+<label x="-116.84" y="0" size="1.778" layer="95"/>
+</segment>
 </net>
 <net name="N$5" class="0">
@@
 </segment>
 </net>
+<net name="N$10" class="0">
+<segment>
+<pinref part="PWM9" gate="A" pin="3"/>
+<wire x1="-129.54" y1="55.88" x2="-93.98" y2="55.88" width="0.1524" layer="91"/>
+<wire x1="-93.98" y1="55.88" x2="-93.98" y2="25.4" width="0.1524" layer="91"/>
+<pinref part="FLIGHTCONTROL" gate="G$1" pin="20/A6/PWM"/>
+<wire x1="-93.98" y1="25.4" x2="-78.74" y2="25.4" width="0.1524" layer="91"/>
+</segment>
+</net>
+<net name="N$11" class="0">
+<segment>
+<pinref part="PWM8" gate="A" pin="3"/>
+<wire x1="-129.54" y1="38.1" x2="-96.52" y2="38.1" width="0.1524" layer="91"/>
+<wire x1="-96.52" y1="38.1" x2="-96.52" y2="22.86" width="0.1524" layer="91"/>
+<pinref part="FLIGHTCONTROL" gate="G$1" pin="21/A7/PWM"/>
+<wire x1="-96.52" y1="22.86" x2="-78.74" y2="22.86" width="0.1524" layer="91"/>
+</segment>
+</net>
+<net name="N$12" class="0">
+<segment>
+<pinref part="PWM7" gate="A" pin="3"/>
+<pinref part="FLIGHTCONTROL" gate="G$1" pin="22/A8/T/PWM"/>
+<wire x1="-129.54" y1="20.32" x2="-78.74" y2="20.32" width="0.1524" layer="91"/>
+</segment>
+</net>
+<net name="N$13" class="0">
+<segment>
+<pinref part="PWM6" gate="A" pin="3"/>
+<wire x1="-129.54" y1="2.54" x2="-96.52" y2="2.54" width="0.1524" layer="91"/>
+<wire x1="-96.52" y1="2.54" x2="-96.52" y2="17.78" width="0.1524" layer="91"/>
+<pinref part="FLIGHTCONTROL" gate="G$1" pin="23/A9/T/PWM"/>
+<wire x1="-96.52" y1="17.78" x2="-78.74" y2="17.78" width="0.1524" layer="91"/>
+</segment>
+</net>

Commit message: finished the schematic i think
Parts:
- added FA, RA: Blue, led:LEDCHIP-LED0603
- added FB: Red, led:LEDCHIP-LED0603
- added R3, R4: 100, resistor:R-US_R0603
- added R6: 150, resistor:R-US_R0603
Connections:
- new net N$14: FLIGHTCONTROL.15/A1/T, R4.1
- new net N$15: FA.A, R4.2
- new net N$16: R3.1, RECEIVER.15/A1/T
- new net N$17: R3.2, RA.A
- new net N$18: FLIGHTCONTROL.16/A2/T, R6.1
- new net N$19: FB.A, R6.2
- net GND: now also FA.C, FB.C, I2C1.1, I2C2.1, I2C3.1, I2C4.1, I2C5.1, RA.C
- net SCL/SCLK: now also I2C1.3, I2C2.3, I2C3.3, I2C4.3, I2C5.3
- net SDA/SDI: now also I2C1.2, I2C2.2, I2C3.2, I2C4.2, I2C5.2
Changed lines of the file:
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@@
 <part name="I2C4" library="pinhead" deviceset="PINHD-1X3" device="" value="GND-SDA-SCL"/>
 <part name="I2C5" library="pinhead" deviceset="PINHD-1X3" device="" value="GND-SDA-SCL"/>
+<part name="U$4" library="Power or GND " deviceset="GND_POWER" device=""/>
+<part name="FA" library="led" deviceset="LED" device="CHIP-LED0603" value="Blue"/>
+<part name="FB" library="led" deviceset="LED" device="CHIP-LED0603" value="Red"/>
+<part name="RA" library="led" deviceset="LED" device="CHIP-LED0603" value="Blue"/>
+<part name="R3" library="resistor" deviceset="R-US_" device="R0603" value="100"/>
+<part name="R4" library="resistor" deviceset="R-US_" device="R0603" value="100"/>
+<part name="U$15" library="Power or GND " deviceset="GND_POWER" device=""/>
+<part name="R6" library="resistor" deviceset="R-US_" device="R0603" value="150"/>
 </parts>
 <sheets>
@@
 <instance part="I2C4" gate="A" x="154.94" y="157.48" rot="R90"/>
 <instance part="I2C5" gate="A" x="172.72" y="157.48" rot="R90"/>
+<instance part="U$4" gate="G$1" x="99.06" y="137.16" rot="R270"/>
+<instance part="FA" gate="G$1" x="-124.46" y="86.36" rot="R270"/>
+<instance part="FB" gate="G$1" x="-124.46" y="76.2" rot="R270"/>
+<instance part="RA" gate="G$1" x="-116.84" y="121.92" rot="R270"/>
+<instance part="R3" gate="G$1" x="-104.14" y="121.92" rot="R180"/>
+<instance part="R4" gate="G$1" x="-111.76" y="86.36" rot="R180"/>
+<instance part="U$15" gate="G$1" x="-149.86" y="127" rot="R180"/>
+<instance part="R6" gate="G$1" x="-111.76" y="76.2" rot="R180"/>
 </instances>
 <busses>
@@
 <label x="-154.94" y="25.4" size="1.778" layer="95"/>
 </segment>
+<segment>
+<pinref part="I2C1" gate="A" pin="1"/>
+<wire x1="99.06" y1="154.94" x2="99.06" y2="137.16" width="0.1524" layer="91"/>
+<pinref part="I2C5" gate="A" pin="1"/>
+<wire x1="99.06" y1="137.16" x2="116.84" y2="137.16" width="0.1524" layer="91"/>
+<wire x1="116.84" y1="137.16" x2="134.62" y2="137.16" width="0.1524" layer="91"/>
+<wire x1="134.62" y1="137.16" x2="152.4" y2="137.16" width="0.1524" layer="91"/>
+<wire x1="152.4" y1="137.16" x2="170.18" y2="137.16" width="0.1524" layer="91"/>
+<wire x1="170.18" y1="137.16" x2="170.18" y2="154.94" width="0.1524" layer="91"/>
+<pinref part="I2C2" gate="A" pin="1"/>
+<wire x1="116.84" y1="154.94" x2="116.84" y2="137.16" width="0.1524" layer="91"/>
+<junction x="116.84" y="137.16"/>
+<junction x="134.62" y="137.16"/>
+<junction x="152.4" y="137.16"/>
+<pinref part="I2C3" gate="A" pin="1"/>
+<wire x1="134.62" y1="154.94" x2="134.62" y2="137.16" width="0.1524" layer="91"/>
+<pinref part="I2C4" gate="A" pin="1"/>
+<wire x1="152.4" y1="154.94" x2="152.4" y2="137.16" width="0.1524" layer="91"/>
+<label x="104.14" y="137.16" size="1.778" layer="95"/>
+<pinref part="U$4" gate="G$1" pin="GND"/>
+<junction x="99.06" y="137.16"/>
+</segment>
+<segment>
+<pinref part="RA" gate="G$1" pin="C"/>
+<pinref part="U$15" gate="G$1" pin="GND"/>
+<wire x1="-121.92" y1="121.92" x2="-149.86" y2="121.92" width="0.1524" layer="91"/>
+<wire x1="-149.86" y1="121.92" x2="-149.86" y2="127" width="0.1524" layer="91"/>
+<pinref part="FA" gate="G$1" pin="C"/>
+<wire x1="-129.54" y1="86.36" x2="-149.86" y2="86.36" width="0.1524" layer="91"/>
+<wire x1="-149.86" y1="86.36" x2="-149.86" y2="121.92" width="0.1524" layer="91"/>
+<pinref part="FB" gate="G$1" pin="C"/>
+<wire x1="-129.54" y1="76.2" x2="-149.86" y2="76.2" width="0.1524" layer="91"/>
+<wire x1="-149.86" y1="76.2" x2="-149.86" y2="86.36" width="0.1524" layer="91"/>
+<label x="-149.86" y="114.3" size="1.778" layer="95"/>
+</segment>
 </net>
 <net name="VCC_3V3" class="0">
@@
 <wire x1="-83.82" y1="27.94" x2="-78.74" y2="27.94" width="0.1524" layer="91"/>
 </segment>
+<segment>
+<pinref part="I2C1" gate="A" pin="3"/>
+<wire x1="104.14" y1="154.94" x2="104.14" y2="142.24" width="0.1524" layer="91"/>
+<label x="104.14" y="142.24" size="1.778" layer="95"/>
+</segment>
+<segment>
+<pinref part="I2C2" gate="A" pin="3"/>
+<wire x1="121.92" y1="154.94" x2="121.92" y2="139.7" width="0.1524" layer="91"/>
+<label x="121.92" y="139.7" size="1.778" layer="95"/>
+</segment>
+<segment>
+<pinref part="I2C3" gate="A" pin="3"/>
+<wire x1="139.7" y1="154.94" x2="139.7" y2="142.24" width="0.1524" layer="91"/>
+<label x="139.7" y="142.24" size="1.778" layer="95"/>
+</segment>
+<segment>
+<pinref part="I2C4" gate="A" pin="3"/>
+<wire x1="157.48" y1="154.94" x2="157.48" y2="139.7" width="0.1524" layer="91"/>
+<label x="157.48" y="139.7" size="1.778" layer="95"/>
+</segment>
+<segment>
+<pinref part="I2C5" gate="A" pin="3"/>
+<wire x1="175.26" y1="154.94" x2="175.26" y2="142.24" width="0.1524" layer="91"/>
+<label x="175.26" y="142.24" size="1.778" layer="95"/>
+</segment>
 </net>
 <net name="SDA/SDI" class="0">
@@
 <wire x1="12.7" y1="35.56" x2="12.7" y2="45.72" width="0.1524" layer="91"/>
 </segment>
+<segment>
+<pinref part="I2C1" gate="A" pin="2"/>
+<wire x1="101.6" y1="154.94" x2="101.6" y2="144.78" width="0.1524" layer="91"/>
+<label x="101.6" y="144.78" size="1.778" layer="95" rot="R90"/>
+</segment>
+<segment>
+<pinref part="I2C2" gate="A" pin="2"/>
+<wire x1="119.38" y1="154.94" x2="119.38" y2="144.78" width="0.1524" layer="91"/>
+<label x="119.38" y="144.78" size="1.778" layer="95" rot="R90"/>
+</segment>
+<segment>
+<pinref part="I2C3" gate="A" pin="2"/>
+<wire x1="137.16" y1="154.94" x2="137.16" y2="144.78" width="0.1524" layer="91"/>
+<label x="137.16" y="144.78" size="1.778" layer="95" rot="R90"/>
+</segment>
+<segment>
+<pinref part="I2C4" gate="A" pin="2"/>
+<wire x1="154.94" y1="154.94" x2="154.94" y2="144.78" width="0.1524" layer="91"/>
+<label x="154.94" y="144.78" size="1.778" layer="95" rot="R90"/>
+</segment>
+<segment>
+<pinref part="I2C5" gate="A" pin="2"/>
+<wire x1="172.72" y1="154.94" x2="172.72" y2="144.78" width="0.1524" layer="91"/>
+<label x="172.72" y="144.78" size="1.778" layer="95" rot="R90"/>
+</segment>
 </net>
 <net name="AD0/SDO" class="0">
@@
 </segment>
 </net>
+<net name="N$14" class="0">
+<segment>
+<pinref part="FLIGHTCONTROL" gate="G$1" pin="15/A1/T"/>
+<wire x1="-78.74" y1="38.1" x2="-88.9" y2="38.1" width="0.1524" layer="91"/>
+<wire x1="-88.9" y1="38.1" x2="-88.9" y2="81.28" width="0.1524" layer="91"/>
+<wire x1="-88.9" y1="81.28" x2="-101.6" y2="81.28" width="0.1524" layer="91"/>
+<wire x1="-101.6" y1="81.28" x2="-101.6" y2="86.36" width="0.1524" layer="91"/>
+<pinref part="R4" gate="G$1" pin="1"/>
+<wire x1="-101.6" y1="86.36" x2="-106.68" y2="86.36" width="0.1524" layer="91"/>
+</segment>
+</net>
+<net name="N$15" class="0">
+<segment>
+<pinref part="R4" gate="G$1" pin="2"/>
+<pinref part="FA" gate="G$1" pin="A"/>
+<wire x1="-116.84" y1="86.36" x2="-121.92" y2="86.36" width="0.1524" layer="91"/>
+</segment>
+</net>
+<net name="N$16" class="0">
+<segment>
+<pinref part="RECEIVER" gate="G$1" pin="15/A1/T"/>
+<pinref part="R3" gate="G$1" pin="1"/>
+<wire x1="-78.74" y1="121.92" x2="-99.06" y2="121.92" width="0.1524" layer="91"/>
+</segment>
+</net>
+<net name="N$17" class="0">
+<segment>
+<pinref part="R3" gate="G$1" pin="2"/>
+<pinref part="RA" gate="G$1" pin="A"/>
+<wire x1="-109.22" y1="121.92" x2="-114.3" y2="121.92" width="0.1524" layer="91"/>
+</segment>
+</net>
+<net name="N$18" class="0">
+<segment>
+<pinref part="R6" gate="G$1" pin="1"/>
+<wire x1="-106.68" y1="76.2" x2="-91.44" y2="76.2" width="0.1524" layer="91"/>
+<wire x1="-91.44" y1="76.2" x2="-91.44" y2="35.56" width="0.1524" layer="91"/>
+<pinref part="FLIGHTCONTROL" gate="G$1" pin="16/A2/T"/>
+<wire x1="-91.44" y1="35.56" x2="-78.74" y2="35.56" width="0.1524" layer="91"/>
+</segment>
+</net>
+<net name="N$19" class="0">
+<segment>
+<pinref part="R6" gate="G$1" pin="2"/>
+<pinref part="FB" gate="G$1" pin="A"/>
+<wire x1="-116.84" y1="76.2" x2="-121.92" y2="76.2" width="0.1524" layer="91"/>
+</segment>
+</net>
