File: Hardware/Teensy-FC-BOB/Teensy-FC-BOB.brd (EAGLE design)
At the start: 100 x 80 mm, 21 parts, among them U1 MPU-9250, U3 BMP180;314030004

Commit message: finishing pins
Parts:
- added I2C1, I2C2, I2C3, I2C4, I2C5: GND-SDA-SCL, pinhead:1X03
- added PWM6: PWMOUT4, pinhead:1X03
- added PWM7: PWMOUT3, pinhead:1X03
- added PWM8: PWMOUT2, pinhead:1X03
- added PWM9: PWMOUT1, pinhead:1X03
Connections:
- new net N$10: FLIGHTCONTROL.20/A6, PWM9.3
- new net N$11: FLIGHTCONTROL.21/A7, PWM8.3
- new net N$12: FLIGHTCONTROL.22/A8, PWM7.3
- new net N$13: FLIGHTCONTROL.23/A9, PWM6.3
- net GND: now also PWM6.1, PWM7.1, PWM8.1, PWM9.1
- net VCC_5V: now also PWM6.2, PWM7.2, PWM8.2, PWM9.2
Changed lines of the file:
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@@
 <element name="PWM5" library="pinhead" package="1X03" value="PWM5" x="-74.93" y="-39.37"/>
 <element name="5V" library="pinhead" package="1X02" value="5V" x="-76.2" y="-46.99"/>
+<element name="PWM6" library="pinhead" package="1X03" value="PWMOUT4" x="-74.93" y="-54.61"/>
+<element name="PWM7" library="pinhead" package="1X03" value="PWMOUT3" x="-74.93" y="-62.23"/>
+<element name="PWM8" library="pinhead" package="1X03" value="PWMOUT2" x="-74.93" y="-69.85"/>
+<element name="PWM9" library="pinhead" package="1X03" value="PWMOUT1" x="-74.93" y="-77.47"/>
+<element name="I2C1" library="pinhead" package="1X03" value="GND-SDA-SCL" x="-74.93" y="-85.09"/>
+<element name="I2C2" library="pinhead" package="1X03" value="GND-SDA-SCL" x="-74.93" y="-92.71"/>
+<element name="I2C3" library="pinhead" package="1X03" value="GND-SDA-SCL" x="-74.93" y="-100.33"/>
+<element name="I2C4" library="pinhead" package="1X03" value="GND-SDA-SCL" x="-74.93" y="-107.95"/>
+<element name="I2C5" library="pinhead" package="1X03" value="GND-SDA-SCL" x="-74.93" y="-115.57"/>
 </elements>
 <signals>
@@
 <contactref element="PWM5" pad="3"/>
 <contactref element="5V" pad="1"/>
+<contactref element="PWM9" pad="1"/>
+<contactref element="PWM8" pad="1"/>
+<contactref element="PWM7" pad="1"/>
+<contactref element="PWM6" pad="1"/>
+<wire x1="-77.47" y1="-69.85" x2="-77.47" y2="-77.47" width="0" layer="19" extent="1-1"/>
+<wire x1="-77.47" y1="-62.23" x2="-77.47" y2="-69.85" width="0" layer="19" extent="1-1"/>
+<wire x1="-77.47" y1="-54.61" x2="-77.47" y2="-62.23" width="0" layer="19" extent="1-1"/>
+<wire x1="-77.47" y1="-46.99" x2="-77.47" y2="-54.61" width="0" layer="19" extent="1-1"/>
 <wire x1="-72.39" y1="-39.37" x2="-77.47" y2="-46.99" width="0" layer="19" extent="1-1"/>
 <wire x1="-72.39" y1="-31.75" x2="-72.39" y2="-39.37" width="0" layer="19" extent="1-1"/>
@@
 <signal name="VCC_5V">
 <contactref element="5V" pad="2"/>
+<contactref element="PWM9" pad="2"/>
+<contactref element="PWM8" pad="2"/>
+<contactref element="PWM7" pad="2"/>
+<contactref element="PWM6" pad="2"/>
+<wire x1="-74.93" y1="-69.85" x2="-74.93" y2="-77.47" width="0" layer="19" extent="1-1"/>
+<wire x1="-74.93" y1="-62.23" x2="-74.93" y2="-69.85" width="0" layer="19" extent="1-1"/>
+<wire x1="-74.93" y1="-54.61" x2="-74.93" y2="-62.23" width="0" layer="19" extent="1-1"/>
+<wire x1="-74.93" y1="-46.99" x2="-74.93" y2="-54.61" width="0" layer="19" extent="1-1"/>
 </signal>
 <signal name="N$5">
@@
 <wire x1="-59.69" y1="20.32" x2="-77.47" y2="-39.37" width="0" layer="19" extent="1-1"/>
 </signal>
+<signal name="N$10">
+<contactref element="PWM9" pad="3"/>
+<contactref element="FLIGHTCONTROL" pad="20/A6"/>
+<wire x1="-63.5" y1="20.32" x2="-72.39" y2="-77.47" width="0" layer="19" extent="1-1"/>
+</signal>
+<signal name="N$11">
+<contactref element="PWM8" pad="3"/>
+<contactref element="FLIGHTCONTROL" pad="21/A7"/>
+<wire x1="-63.5" y1="22.86" x2="-72.39" y2="-69.85" width="0" layer="19" extent="1-1"/>
+</signal>
+<signal name="N$12">
+<contactref element="PWM7" pad="3"/>
+<contactref element="FLIGHTCONTROL" pad="22/A8"/>
+<wire x1="-63.5" y1="25.4" x2="-72.39" y2="-62.23" width="0" layer="19" extent="1-1"/>
+</signal>
+<signal name="N$13">
+<contactref element="PWM6" pad="3"/>
+<contactref element="FLIGHTCONTROL" pad="23/A9"/>
+<wire x1="-63.5" y1="27.94" x2="-72.39" y2="-54.61" width="0" layer="19" extent="1-1"/>
+</signal>
 </signals>

Commit message: finished the schematic i think
Parts:
- added FA, RA: Blue, led:CHIP-LED0603
- added FB: Red, led:CHIP-LED0603
- added R3, R4: 100, resistor:R0603
- added R6: 150, resistor:R0603
Connections:
- new net N$14: FLIGHTCONTROL.15/A1, R4.1
- new net N$15: FA.A, R4.2
- new net N$16: R3.1, RECEIVER.15/A1
- new net N$17: R3.2, RA.A
- new net N$18: FLIGHTCONTROL.16/A2, R6.1
- new net N$19: FB.A, R6.2
- net GND: now also FA.C, FB.C, I2C1.1, I2C2.1, I2C3.1, I2C4.1, I2C5.1, RA.C
- net SCL/SCLK: now also I2C1.3, I2C2.3, I2C3.3, I2C4.3, I2C5.3
- net SDA/SDI: now also I2C1.2, I2C2.2, I2C3.2, I2C4.2, I2C5.2
Changed lines of the file:
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@@
 <element name="I2C4" library="pinhead" package="1X03" value="GND-SDA-SCL" x="-74.93" y="-107.95"/>
 <element name="I2C5" library="pinhead" package="1X03" value="GND-SDA-SCL" x="-74.93" y="-115.57"/>
+<element name="FA" library="led" package="CHIP-LED0603" value="Blue" x="-82.55" y="-116.84"/>
+<element name="FB" library="led" package="CHIP-LED0603" value="Red" x="-87.63" y="-116.84"/>
+<element name="RA" library="led" package="CHIP-LED0603" value="Blue" x="-92.71" y="-116.84"/>
+<element name="R3" library="resistor" package="R0603" value="100" x="-92.71" y="-121.92"/>
+<element name="R4" library="resistor" package="R0603" value="100" x="-92.71" y="-127"/>
+<element name="R6" library="resistor" package="R0603" value="150" x="-92.71" y="-132.08"/>
 </elements>
 <signals>
@@
 <contactref element="PWM7" pad="1"/>
 <contactref element="PWM6" pad="1"/>
+<contactref element="I2C1" pad="1"/>
+<contactref element="I2C5" pad="1"/>
+<contactref element="I2C2" pad="1"/>
+<contactref element="I2C3" pad="1"/>
+<contactref element="I2C4" pad="1"/>
+<contactref element="RA" pad="C"/>
+<contactref element="FA" pad="C"/>
+<contactref element="FB" pad="C"/>
+<wire x1="-87.63" y1="-116.09" x2="-92.71" y2="-116.09" width="0" layer="19" extent="1-1"/>
+<wire x1="-82.55" y1="-116.09" x2="-87.63" y2="-116.09" width="0" layer="19" extent="1-1"/>
+<wire x1="-77.47" y1="-115.57" x2="-82.55" y2="-116.09" width="0" layer="19" extent="1-1"/>
+<wire x1="-77.47" y1="-107.95" x2="-77.47" y2="-115.57" width="0" layer="19" extent="1-1"/>
+<wire x1="-77.47" y1="-100.33" x2="-77.47" y2="-107.95" width="0" layer="19" extent="1-1"/>
+<wire x1="-77.47" y1="-92.71" x2="-77.47" y2="-100.33" width="0" layer="19" extent="1-1"/>
+<wire x1="-77.47" y1="-85.09" x2="-77.47" y2="-92.71" width="0" layer="19" extent="1-1"/>
+<wire x1="-77.47" y1="-77.47" x2="-77.47" y2="-85.09" width="0" layer="19" extent="1-1"/>
 <wire x1="-77.47" y1="-69.85" x2="-77.47" y2="-77.47" width="0" layer="19" extent="1-1"/>
 <wire x1="-77.47" y1="-62.23" x2="-77.47" y2="-69.85" width="0" layer="19" extent="1-1"/>
@@
 <contactref element="R1" pad="1"/>
 <contactref element="FLIGHTCONTROL" pad="19/A5"/>
+<contactref element="I2C1" pad="3"/>
+<contactref element="I2C2" pad="3"/>
+<contactref element="I2C3" pad="3"/>
+<contactref element="I2C4" pad="3"/>
+<contactref element="I2C5" pad="3"/>
+<wire x1="-72.39" y1="-107.95" x2="-72.39" y2="-115.57" width="0" layer="19" extent="1-1"/>
+<wire x1="-72.39" y1="-100.33" x2="-72.39" y2="-107.95" width="0" layer="19" extent="1-1"/>
+<wire x1="-72.39" y1="-92.71" x2="-72.39" y2="-100.33" width="0" layer="19" extent="1-1"/>
+<wire x1="-72.39" y1="-85.09" x2="-72.39" y2="-92.71" width="0" layer="19" extent="1-1"/>
+<wire x1="-78.32" y1="-2.54" x2="-72.39" y2="-85.09" width="0" layer="19" extent="1-1"/>
 <wire x1="-63.5" y1="17.78" x2="-78.32" y2="-2.54" width="0" layer="19" extent="1-1"/>
 <wire x1="-34.89" y1="20.65" x2="-63.5" y2="17.78" width="0" layer="19" extent="1-1"/>
@@
 <contactref element="R2" pad="2"/>
 <contactref element="FLIGHTCONTROL" pad="18/A4"/>
+<contactref element="I2C1" pad="2"/>
+<contactref element="I2C2" pad="2"/>
+<contactref element="I2C3" pad="2"/>
+<contactref element="I2C4" pad="2"/>
+<contactref element="I2C5" pad="2"/>
+<wire x1="-74.93" y1="-107.95" x2="-74.93" y2="-115.57" width="0" layer="19" extent="1-1"/>
+<wire x1="-74.93" y1="-100.33" x2="-74.93" y2="-107.95" width="0" layer="19" extent="1-1"/>
+<wire x1="-74.93" y1="-92.71" x2="-74.93" y2="-100.33" width="0" layer="19" extent="1-1"/>
+<wire x1="-74.93" y1="-85.09" x2="-74.93" y2="-92.71" width="0" layer="19" extent="1-1"/>
+<wire x1="-76.62" y1="-6.35" x2="-74.93" y2="-85.09" width="0" layer="19" extent="1-1"/>
 <wire x1="-63.5" y1="15.24" x2="-76.62" y2="-6.35" width="0" layer="19" extent="1-1"/>
 <wire x1="-35.29" y1="20.65" x2="-63.5" y2="15.24" width="0" layer="19" extent="1-1"/>
@@
 <wire x1="-63.5" y1="27.94" x2="-72.39" y2="-54.61" width="0" layer="19" extent="1-1"/>
 </signal>
+<signal name="N$14">
+<contactref element="FLIGHTCONTROL" pad="15/A1"/>
+<contactref element="R4" pad="1"/>
+<wire x1="-63.5" y1="7.62" x2="-93.56" y2="-127" width="0" layer="19" extent="1-1"/>
+</signal>
+<signal name="N$15">
+<contactref element="R4" pad="2"/>
+<contactref element="FA" pad="A"/>
+<wire x1="-82.55" y1="-117.59" x2="-91.86" y2="-127" width="0" layer="19" extent="1-1"/>
+</signal>
+<signal name="N$16">
+<contactref element="RECEIVER" pad="15/A1"/>
+<contactref element="R3" pad="1"/>
+<wire x1="-44.45" y1="7.62" x2="-93.56" y2="-121.92" width="0" layer="19" extent="1-1"/>
+</signal>
+<signal name="N$17">
+<contactref element="R3" pad="2"/>
+<contactref element="RA" pad="A"/>
+<wire x1="-92.71" y1="-117.59" x2="-91.86" y2="-121.92" width="0" layer="19" extent="1-1"/>
+</signal>
+<signal name="N$18">
+<contactref element="R6" pad="1"/>
+<contactref element="FLIGHTCONTROL" pad="16/A2"/>
+<wire x1="-63.5" y1="10.16" x2="-93.56" y2="-132.08" width="0" layer="19" extent="1-1"/>
+</signal>
+<signal name="N$19">
+<contactref element="R6" pad="2"/>
+<contactref element="FB" pad="A"/>
+<wire x1="-87.63" y1="-117.59" x2="-91.86" y2="-132.08" width="0" layer="19" extent="1-1"/>
+</signal>
 </signals>

Commit message: started the board layout
Parts:
- moved R2 119.0 mm to (36.8, 26.7), turned to 180 degrees
- moved R1 117.4 mm to (36.8, 24.1)
- moved INT 113.1 mm to (71.1, 36.8)
- moved FLIGHTCONTROL 109.3 mm to (38.1, 22.9), turned to 180 degrees
- moved C10 98.0 mm to (62.2, 35.6)
- moved C8 96.1 mm to (64.8, 41.9)
- moved U1 91.2 mm to (54.6, 39.4)
- moved C7 90.9 mm to (59.7, 39.4)
- moved C5 90.4 mm to (49.5, 35.6)
- moved C9 86.0 mm to (58.4, 43.2)
- moved C6 85.7 mm to (59.7, 30.5)
- moved U3 76.0 mm to (54.6, 31.8)
- moved RECEIVER 68.7 mm to (16.5, 22.9), turned to 180 degrees
- moved R5 64.8 mm to (49.5, 43.2)
- moved ADDR 57.4 mm to (39.4, 43.2), turned to 180 degrees
Other:
- board size 100 x 80 mm -> 75.9 x 45.7 mm

Commit message: routing wires
Parts:
- moved R6 205.9 mm to (59.7, 6.35)
- moved R4 199.7 mm to (55.9, 6.35)
- moved I2C5 194.4 mm to (71.1, 12.7)
- moved R3 192.5 mm to (50.8, 6.35)
- moved I2C4 191.9 mm to (71.1, 16.5)
- moved FB 189.6 mm to (59.7, 2.54), turned to 180 degrees
- moved I2C3 189.4 mm to (71.1, 20.3)
- moved I2C2 187.0 mm to (71.1, 24.1)
- moved RA 186.7 mm to (50.8, 2.54), turned to 180 degrees
- moved I2C1 184.7 mm to (71.1, 27.9)
- moved FA 183.8 mm to (57.1, 2.54), turned to 180 degrees
- moved PWM9 166.3 mm to (62.2, 16.5)
- moved PWM8 164.1 mm to (62.2, 20.3)
- moved PWM7 162.1 mm to (62.2, 24.1)
- moved PWM6 160.1 mm to (62.2, 27.9)
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Routing:
- net GND: track 0.00 -> 238.3 mm
- net VCC_3V3: track 0.00 -> 139.8 mm, vias 0 -> 1
- net SCL/SCLK: track 0.00 -> 79.0 mm, vias 0 -> 2
- net N$6: track 0.00 -> 74.2 mm
- net N$16: track 0.00 -> 68.9 mm
- net SDA/SDI: track 0.00 -> 68.1 mm, vias 0 -> 2
- net N$14: track 0.00 -> 56.1 mm
- net N$5: track 0.00 -> 52.8 mm
- net N$13: track 0.00 -> 50.3 mm
- net N$8: track 0.00 -> 47.7 mm, vias 0 -> 1
- net N$18: track 0.00 -> 47.2 mm, vias 0 -> 1
- net N$11: track 0.00 -> 47.2 mm, vias 0 -> 2
- net N$7: track 0.00 -> 44.0 mm
- net N$12: track 0.00 -> 43.9 mm
- net N$10: track 0.00 -> 39.6 mm
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
Commit message: finished routing
Routing:
- net VCC_3V3: track 139.8 -> 163.3 mm, vias 1 -> 3
- net SCL/SCLK: track 79.0 -> 97.0 mm, vias 2 -> 4
- net AD0/SDO: track 0.00 -> 15.7 mm, vias 0 -> 2
- net SDA/SDI: track 68.1 -> 80.9 mm, vias 2 -> 3
- net N$4: track 4.89 -> 10.7 mm, vias 0 -> 2
- net GND: track 238.3 -> 243.5 mm
- net N$3: track 0.00 -> 2.80 mm
Other:
- board size 75.9 x 45.7 mm -> 75.9 x 47 mm
