File: Hardware/Teensy-FC-BOB/Teensy-FC-BOB.brd (EAGLE design)
At the start: 75.9 x 47 mm, 36 parts, among them U1 MPU-9250, U3 BMP180;314030004

Commit message: checked around the cpu
Routing:
- net GND: track 243.5 -> 245.3 mm
Changed lines of the file:
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@@
 <wire x1="24.2316" y1="6.1722" x2="24.13" y2="6.35" width="0.254" layer="16"/>
 <wire x1="45.72" y1="6.1722" x2="45.72" y2="6.35" width="0.254" layer="16"/>
-<wire x1="57.6072" y1="41.8338" x2="56.5912" y2="40.8178" width="0.254" layer="1"/>
-<wire x1="56.5912" y1="40.8178" x2="56.4642" y2="40.6908" width="0.254" layer="1"/>
-<wire x1="56.4642" y1="40.6908" x2="56.2356" y2="40.4622" width="0.254" layer="1"/>
-<wire x1="56.2356" y1="40.4622" x2="56.21" y2="40.37" width="0.254" layer="1"/>
-<wire x1="57.6072" y1="41.8338" x2="57.658" y2="41.91" width="0.254" layer="1"/>
 <wire x1="53.721" y1="34.29" x2="51.562" y2="34.29" width="0.254" layer="1"/>
 <wire x1="54.4068" y1="33.6042" x2="53.721" y2="34.29" width="0.254" layer="1"/>
@@
 <wire x1="57.15" y1="44.3484" x2="57.15" y2="44.45" width="0.254" layer="1"/>
 <wire x1="51.435" y1="34.29" x2="51.562" y2="34.29" width="0.254" layer="1"/>
-<wire x1="56.9214" y1="40.2336" x2="56.4642" y2="40.6908" width="0.254" layer="1"/>
-<wire x1="56.9214" y1="35.8902" x2="56.9214" y2="40.2336" width="0.254" layer="1"/>
 <wire x1="54.6354" y1="33.6042" x2="56.1721" y2="35.1409" width="0.254" layer="1"/>
-<wire x1="56.1721" y1="35.1409" x2="56.9214" y2="35.8902" width="0.254" layer="1"/>
 <wire x1="54.6354" y1="33.6042" x2="54.61" y2="33.528" width="0.254" layer="1"/>
 <wire x1="56.007" y1="27.8892" x2="56.007" y2="24.2316" width="0.254" layer="1"/>
@@
 <wire x1="48.26" y1="43.18" x2="48.26" y2="41.402" width="0.3048" layer="1"/>
 <wire x1="48.26" y1="41.402" x2="48.2346" y2="41.3766" width="0.3048" layer="1"/>
-<wire x1="55.21" y1="40.97" x2="55.21" y2="41.367" width="0.254" layer="1"/>
-<wire x1="55.21" y1="41.367" x2="55.499" y2="41.656" width="0.254" layer="1"/>
-<wire x1="55.499" y1="41.656" x2="55.753" y2="41.656" width="0.254" layer="1"/>
-<wire x1="55.753" y1="41.656" x2="56.5912" y2="40.8178" width="0.254" layer="1"/>
+<wire x1="55.21" y1="41.367" x2="55.753" y2="41.91" width="0.254" layer="1"/>
 <wire x1="55.21" y1="37.77" x2="55.21" y2="36.103" width="0.254" layer="1"/>
 <wire x1="55.21" y1="36.103" x2="56.1721" y2="35.1409" width="0.254" layer="1"/>
+<wire x1="55.21" y1="40.97" x2="55.21" y2="41.367" width="0.254" layer="1"/>
+<wire x1="55.753" y1="41.91" x2="57.658" y2="41.91" width="0.254" layer="1"/>
+<wire x1="57.658" y1="41.91" x2="57.658" y2="41.021" width="0.254" layer="1"/>
+<wire x1="57.658" y1="41.021" x2="57.023" y2="40.386" width="0.254" layer="1"/>
+<wire x1="57.023" y1="40.386" x2="56.226" y2="40.386" width="0.254" layer="1"/>
+<wire x1="56.226" y1="40.386" x2="56.21" y2="40.37" width="0.254" layer="1"/>
+<wire x1="57.658" y1="36.6268" x2="56.1721" y2="35.1409" width="0.254" layer="1"/>
+<wire x1="57.658" y1="36.6268" x2="57.658" y2="41.021" width="0.254" layer="1"/>
 </signal>
 <signal name="VCC_3V3">
